File: and.kicad_sch (KiCad schematic)
At the start: 4 parts, among them Q21 DMP3099L, Q22 2N7002, Q23 2N7002, Q24 DMP3099L

Commit message: added decoupling caps
Parts:
- added C35: 10n, symbol Device:C
Connections:
- net GND: now also C35.2
- net VDD renamed +3V3
- net +3V3: now also C35.1

Commit message: corrected output/input type of pins
Parts:
- C16: renamed from C35; footprint (none) -> Capacitor_SMD:C_0603_1608Metric
