File: nand4.kicad_sch (KiCad schematic)
At the start: 8 parts, among them Q549 DMP3099L, Q550 DMP3099L, Q551 2N7002, Q552 2N7002, Q553 2N7002, Q554 2N7002, Q555 DMP3099L, Q556 DMP3099L

Commit message: added decoupling caps
Connections:
- net VDD renamed +3V3
Changed lines of the file:
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@@
+	)
+	(junction
+		(at 154.94 85.09)
+		(diameter 0)
+		(color 0 0 0 0)
+	)
+	(junction
+		(at 166.37 74.93)
+		(diameter 0)
+		(color 0 0 0 0)
+	)
+	(junction
+		(at 142.24 74.93)
+		(diameter 0)
+		(color 0 0 0 0)
+	)
+	(junction
+		(at 166.37 85.09)
+		(diameter 0)
+		(color 0 0 0 0)
+	)
+	(junction
+		(at 154.94 87.63)
+		(diameter 0)
+		(color 0 0 0 0)
 	)
 	(junction
@@
 		(color 0 0 0 0)
 	)
-	(junction
-		(at 154.94 85.09)
-		(diameter 0)
-		(color 0 0 0 0)
-	)
-	(junction
-		(at 166.37 74.93)
-		(diameter 0)
-		(color 0 0 0 0)
-	)
-	(junction
-		(at 142.24 74.93)
-		(diameter 0)
-		(color 0 0 0 0)
-	)
-	(junction
-		(at 166.37 85.09)
-		(diameter 0)
-		(color 0 0 0 0)
-	)
-	(junction
-		(at 154.94 87.63)
-		(diameter 0)
-		(color 0 0 0 0)
-	)
 	(wire
 		(pts
@@
 	(wire
 		(pts
+			(xy 118.11 74.93) (xy 142.24 74.93)
+		)
+		(stroke
+			(width 0)
+			(type default)
+		)
+	)
+	(wire
+		(pts
+			(xy 142.24 85.09) (xy 154.94 85.09)
+		)
+		(stroke
+			(width 0)
+			(type default)
+		)
+	)
+	(wire
+		(pts
+			(xy 154.94 87.63) (xy 154.94 90.17)
+		)
+		(stroke
+			(width 0)
+			(type default)
+		)
+	)
+	(wire
+		(pts
+			(xy 154.94 85.09) (xy 154.94 87.63)
+		)
+		(stroke
+			(width 0)
+			(type default)
+		)
+	)
+	(wire
+		(pts
+			(xy 166.37 85.09) (xy 190.5 85.09)
+		)
+		(stroke
+			(width 0)
+			(type default)
+		)
+	)
+	(wire
+		(pts
+			(xy 154.94 124.46) (xy 154.94 128.27)
+		)
+		(stroke
+			(width 0)
+			(type default)
+		)
+	)
+	(wire
+		(pts
+			(xy 118.11 85.09) (xy 142.24 85.09)
+		)
+		(stroke
+			(width 0)
+			(type default)
+		)
+	)
+	(wire
+		(pts
+			(xy 142.24 74.93) (xy 154.94 74.93)
+		)
+		(stroke
+			(width 0)
+			(type default)
+		)
+	)
+	(wire
+		(pts
 			(xy 154.94 74.93) (xy 166.37 74.93)
-		)
-		(stroke
-			(width 0)
-			(type default)
-		)
-	)
-	(wire
-		(pts
-			(xy 118.11 74.93) (xy 142.24 74.93)
-		)
-		(stroke
-			(width 0)
-			(type default)
-		)
-	)
-	(wire
-		(pts
-			(xy 142.24 85.09) (xy 154.94 85.09)
-		)
-		(stroke
-			(width 0)
-			(type default)
-		)
-	)
-	(wire
-		(pts
-			(xy 154.94 87.63) (xy 154.94 90.17)
-		)
-		(stroke
-			(width 0)
-			(type default)
-		)
-	)
-	(wire
-		(pts
-			(xy 154.94 85.09) (xy 154.94 87.63)
-		)
-		(stroke
-			(width 0)
-			(type default)
-		)
-	)
-	(wire
-		(pts
-			(xy 166.37 85.09) (xy 190.5 85.09)
-		)
-		(stroke
-			(width 0)
-			(type default)
-		)
-	)
-	(wire
-		(pts
-			(xy 154.94 124.46) (xy 154.94 128.27)
-		)
-		(stroke
-			(width 0)
-			(type default)
-		)
-	)
-	(wire
-		(pts
-			(xy 118.11 85.09) (xy 142.24 85.09)
-		)
-		(stroke
-			(width 0)
-			(type default)
-		)
-	)
-	(wire
-		(pts
-			(xy 142.24 74.93) (xy 154.94 74.93)
 		)
 		(stroke
@@
 	)
 	(symbol
-		(lib_id "power:VDD")
+		(lib_id "power:+3V3")
 		(at 154.94 74.93 0)
 		(unit 1)
@@
 			)
 		)
-		(property "Value" "VDD"
+		(property "Value" "+3V3"
 			(at 154.94 70.7969 0)
 			(effects
@@
 			)
 		)
-		(property "Description" "Power symbol creates a global label with name \"VDD\""
+		(property "Description" "Power symbol creates a global label with name \"+3V3\""
 			(at 154.94 74.93 0)
 			(effects

Commit message: corrected output/input type of pins
Parts:
- renumbered Q549 to Q591, Q550 to Q592, Q551 to Q593, Q552 to Q594, Q553 to Q595, Q554 to Q596, Q555 to Q597, Q556 to Q598

Commit message: schematic cleanup, routed 1 bdc
Parts:
- renumbered Q591 to Q639, Q592 to Q640, Q593 to Q641, Q594 to Q642, Q595 to Q643, Q596 to Q644, Q597 to Q645, Q598 to Q646
