File: nand3.kicad_sch (KiCad schematic)
At the start: 6 parts, among them Q29 DMP3099L, Q30 2N7002, Q31 2N7002, Q32 2N7002, Q33 DMP3099L, Q34 DMP3099L

Commit message: added decoupling caps
Connections:
- net VDD renamed +3V3

Commit message: corrected output/input type of pins
Parts:
- renumbered Q29 to Q61, Q30 to Q62, Q31 to Q63, Q32 to Q64, Q33 to Q65, Q34 to Q66

Commit message: schematic cleanup, routed 1 bdc
Parts:
- renumbered Q61 to Q107, Q62 to Q108, Q63 to Q109, Q64 to Q110, Q65 to Q111, Q66 to Q112

Commit message: replace bcd logic with bin-to-dec module
Parts:
- renumbered Q107 to Q87, Q108 to Q88, Q109 to Q89, Q110 to Q90, Q111 to Q91, Q112 to Q92

Commit message: switched to using flipflop module
Parts:
- renumbered Q87 to Q201, Q88 to Q202, Q89 to Q203, Q90 to Q204, Q91 to Q205, Q92 to Q206
