File: bdc.kicad_sch (KiCad schematic)
At the start: 3 parts

Commit message: added footprints for modules
Parts:
- U17: renamed from U3; footprint (none) -> custom:module_bdc_mpcie
- renumbered C40 to C23, C41 to C24

Commit message: added module for PSU
Parts:
- U11: renamed from U17; value ~ -> bin-to-dec; LCSC Part # (none) -> C185937

Commit message: routy mcRouteface
Parts:
- C23, C24: LCSC Part # C57112 -> C19702
Changed lines of the file:
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@@
 			)
 		)
-		(property "LCSC Part #" "C57112"
+		(property "LCSC Part #" "C19702"
 			(at 166.37 104.14 0)
 			(effects
@@
 			)
 		)
-		(property "LCSC Part #" "C57112"
+		(property "LCSC Part #" "C19702"
 			(at 156.21 104.14 0)
 			(effects
