File: counters.kicad_sch (KiCad schematic)
At the start: 22 parts, among them J10 Conn_01x10_Socket, J11 Conn_01x06_Socket, J12 Conn_01x10_Socket, J13 Conn_01x03_Socket, J8 Conn_01x10_Socket, J9 Conn_01x06_Socket, SW1 MIN +, SW2 HR +, U3 SSR, U8 bin-to-dec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

Commit message: routing
Parts:
- J10, J11, J12, J13, J8, J9: now left out of the parts list
Other:
- moved on the sheet: J8
Changed lines of the file:
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@@
 	(wire
 		(pts
-			(xy 12.7 64.77) (xy 12.7 62.23)
-		)
-		(stroke
-			(width 0)
-			(type default)
-		)
-	)
-	(wire
-		(pts
 			(xy 209.55 130.81) (xy 217.17 130.81)
 		)
@@
 	(wire
 		(pts
-			(xy 97.79 64.77) (xy 97.79 62.23)
-		)
-		(stroke
-			(width 0)
-			(type default)
-		)
-	)
-	(wire
-		(pts
 			(xy 121.92 105.41) (xy 119.38 105.41)
 		)
@@
 	(wire
 		(pts
-			(xy 177.8 66.04) (xy 177.8 63.5)
-		)
-		(stroke
-			(width 0)
-			(type default)
-		)
-	)
-	(wire
-		(pts
 			(xy 42.8625 71.12) (xy 42.8625 77.47)
 		)
@@
 	(hierarchical_label "Sqr1"
 		(shape input)
-		(at 12.7 62.23 90)
+		(at 12.7 64.77 270)
 		(effects
 			(font
 				(size 1.27 1.27)
 			)
-			(justify left)
+			(justify right)
 		)
 	)
 	(hierarchical_label "Sqr1"
 		(shape input)
-		(at 177.8 63.5 90)
+		(at 177.8 66.04 270)
 		(effects
 			(font
 				(size 1.27 1.27)
 			)
-			(justify left)
+			(justify right)
 		)
 	)
@@
 	(hierarchical_label "Sqr1"
 		(shape input)
-		(at 97.79 62.23 90)
+		(at 97.79 64.77 180)
 		(effects
 			(font
 				(size 1.27 1.27)
 			)
-			(justify left)
+			(justify right)
 		)
 	)
@@
 		(unit 1)
 		(exclude_from_sim no)
-		(in_bom yes)
+		(in_bom no)
 		(on_board yes)
 		(dnp no)
@@
 		(unit 1)
 		(exclude_from_sim no)
-		(in_bom yes)
+		(in_bom no)
 		(on_board yes)
 		(dnp no)
@@
 		(unit 1)
 		(exclude_from_sim no)
-		(in_bom yes)
+		(in_bom no)
 		(on_board yes)
 		(dnp no)
@@
 		(unit 1)
 		(exclude_from_sim no)
-		(in_bom yes)
+		(in_bom no)
 		(on_board yes)
 		(dnp no)
@@
 		(unit 1)
 		(exclude_from_sim no)
-		(in_bom yes)
+		(in_bom no)
 		(on_board yes)
 		(dnp no)
@@
 	(symbol
 		(lib_id "Connector:Conn_01x10_Socket")
-		(at 30.1625 52.07 90)
+		(at 29.21 52.07 90)
 		(unit 1)
 		(exclude_from_sim no)
-		(in_bom yes)
+		(in_bom no)
 		(on_board yes)
 		(dnp no)
 		(fields_autoplaced yes)
 		(property "Reference" "J8"
-			(at 31.4325 47.9763 90)
+			(at 30.48 47.9763 90)
 			(effects
 				(font
@@
 		)
 		(property "Value" "Conn_01x10_Socket"
-			(at 31.4325 50.4006 90)
+			(at 30.48 50.4006 90)
 			(effects
 				(font
@@
 		)
 		(property "Footprint" "Connector_PinHeader_2.54mm:PinHeader_1x10_P2.54mm_Vertical"
-			(at 30.1625 52.07 0)
+			(at 29.21 52.07 0)
 			(effects
 				(font
@@
 		)
 		(property "Datasheet" "~"
-			(at 30.1625 52.07 0)
+			(at 29.21 52.07 0)
 			(effects
 				(font
@@
 		)
 		(property "Description" "Generic connector, single row, 01x10, script generated"
-			(at 30.1625 52.07 0)
+			(at 29.21 52.07 0)
 			(effects
 				(font
@@
 		)
 		(property "LCSC Part #" ""
-			(at 30.1625 52.07 90)
+			(at 29.21 52.07 90)
 			(effects
 				(font
@@
 		)
 		(pin "Out0" output
-			(at 20.0025 57.15 90)
+			(at 19.05 57.15 90)
 			(effects
 				(font
@@
 		)
 		(pin "Out1" output
-			(at 22.5425 57.15 90)
+			(at 21.59 57.15 90)
 			(effects
 				(font
@@
 		)
 		(pin "Out2" output
-			(at 25.0825 57.15 90)
+			(at 24.13 57.15 90)
 			(effects
 				(font
@@
 		)
 		(pin "Out3" output
-			(at 27.6225 57.15 90)
+			(at 26.67 57.15 90)
 			(effects
 				(font
@@
 		)
 		(pin "Out4" output
-			(at 30.1625 57.15 90)
+			(at 29.21 57.15 90)
 			(effects
 				(font
@@
 		)
 		(pin "Out5" output
-			(at 32.7025 57.15 90)
+			(at 31.75 57.15 90)
 			(effects
 				(font
@@
 		)
 		(pin "Out6" output
-			(at 35.2425 57.15 90)
+			(at 34.29 57.15 90)
 			(effects
 				(font
@@
 		)
 		(pin "Out7" output
-			(at 37.7825 57.15 90)
+			(at 36.83 57.15 90)
 			(effects
 				(font
@@
 		)
 		(pin "Out8" output
-			(at 40.3225 57.15 90)
+			(at 39.37 57.15 90)
 			(effects
 				(font
@@
 		)
 		(pin "Out9" output
-			(at 42.8625 57.15 90)
+			(at 41.91 57.15 90)
 			(effects
 				(font

Commit message: flipflop wip
Connections:
- net relays_h1/Out0: now reaches J13.1 (Pin_1), U3.27
- net relays_h1/Out1: now reaches J13.2 (Pin_2), U3.28
- net relays_h1/Out2: now reaches J13.3 (Pin_3), U3.29
Changed lines of the file:
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@@
+		)
+	)
+	(label "relays_h1{slash}Out2"
+		(at 266.7 49.53 0)
+		(effects
+			(font
+				(size 1.27 1.27)
+			)
+			(justify left bottom)
+		)
+	)
+	(label "relays_h1{slash}Out0"
+		(at 246.38 50.8 0)
+		(effects
+			(font
+				(size 1.27 1.27)
+			)
+			(justify left bottom)
+		)
+	)
+	(label "relays_h1{slash}Out1"
+		(at 262.89 53.34 0)
+		(effects
+			(font
+				(size 1.27 1.27)
+			)
+			(justify left bottom)
 		)
 	)
