File: bcd6.kicad_sch (KiCad schematic)
At the start: 1 part

Commit message: added footprints for modules
Parts:
- U11: renamed from U9; footprint (none) -> custom:module_flipflop_mpcie
Changed lines of the file:
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@@
 	)
 	(symbol
-		(lib_name "jk-flipflops_1")
 		(lib_id "custom:jk-flipflops")
 		(at 66.04 105.41 0)
@@
 		(dnp no)
 		(fields_autoplaced yes)
-		(property "Reference" "U9"
-			(at 66.04 105.41 0)
-			(effects
-				(font
-					(size 1.27 1.27)
-				)
+		(property "Reference" "U11"
+			(at 73.2633 105.0869 0)
+			(effects
+				(font
+					(size 1.27 1.27)
+				)
+				(justify left)
 			)
 		)
@@
 			)
 		)
-		(property "Footprint" ""
+		(property "Footprint" "custom:module_flipflop_mpcie"
 			(at 66.04 105.41 0)
 			(effects
@@
 		(pin "8"
 		)
-		(pin "35"
+		(pin "31"
 		)
 		(instances
 			(project "transistor-clock"
 				(path "/ce10d5bc-995e-4952-aa76-0a08f713a0f2/2c36a9e9-de42-4705-9ad4-94f4cc168e2f/45f6b4b3-4b31-405d-8488-938c33278b8a"
-					(reference "U10")
+					(reference "U12")
 					(unit 1)
 				)
 				(path "/ce10d5bc-995e-4952-aa76-0a08f713a0f2/2c36a9e9-de42-4705-9ad4-94f4cc168e2f/6e22859f-9bca-4d3f-9901-b092abdf20a9"
-					(reference "U9")
+					(reference "U11")
 					(unit 1)
 				)
@@
 		(dnp no)
 		(fields_autoplaced yes)
-		(property "Reference" "U9"
-			(at 92.71 105.41 0)
-			(effects
-				(font
-					(size 1.27 1.27)
-				)
+		(property "Reference" "U11"
+			(at 99.9333 105.0869 0)
+			(effects
+				(font
+					(size 1.27 1.27)
+				)
+				(justify left)
 			)
 		)
@@
 			)
 		)
-		(property "Footprint" ""
+		(property "Footprint" "custom:module_flipflop_mpcie"
 			(at 92.71 105.41 0)
 			(effects
@@
 		(pin "8"
 		)
-		(pin "35"
+		(pin "31"
 		)
 		(instances
 			(project "transistor-clock"
 				(path "/ce10d5bc-995e-4952-aa76-0a08f713a0f2/2c36a9e9-de42-4705-9ad4-94f4cc168e2f/45f6b4b3-4b31-405d-8488-938c33278b8a"
-					(reference "U10")
+					(reference "U12")
 					(unit 2)
 				)
 				(path "/ce10d5bc-995e-4952-aa76-0a08f713a0f2/2c36a9e9-de42-4705-9ad4-94f4cc168e2f/6e22859f-9bca-4d3f-9901-b092abdf20a9"
-					(reference "U9")
+					(reference "U11")
 					(unit 2)
 				)
@@
 	)
 	(symbol
-		(lib_name "jk-flipflops_3")
 		(lib_id "custom:jk-flipflops")
 		(at 124.46 105.41 0)
@@
 		(dnp no)
 		(fields_autoplaced yes)
-		(property "Reference" "U9"
-			(at 124.46 105.41 0)
-			(effects
-				(font
-					(size 1.27 1.27)
-				)
+		(property "Reference" "U11"
+			(at 131.6833 105.0869 0)
+			(effects
+				(font
+					(size 1.27 1.27)
+				)
+				(justify left)
 			)
 		)
@@
 			)
 		)
-		(property "Footprint" ""
+		(property "Footprint" "custom:module_flipflop_mpcie"
 			(at 124.46 105.41 0)
 			(effects
@@
 		(pin "8"
 		)
-		(pin "35"
+		(pin "31"
 		)
 		(instances
 			(project "transistor-clock"
 				(path "/ce10d5bc-995e-4952-aa76-0a08f713a0f2/2c36a9e9-de42-4705-9ad4-94f4cc168e2f/45f6b4b3-4b31-405d-8488-938c33278b8a"
-					(reference "U10")
+					(reference "U12")
 					(unit 3)
 				)
 				(path "/ce10d5bc-995e-4952-aa76-0a08f713a0f2/2c36a9e9-de42-4705-9ad4-94f4cc168e2f/6e22859f-9bca-4d3f-9901-b092abdf20a9"
-					(reference "U9")
+					(reference "U11")
 					(unit 3)
 				)
@@
 		(dnp no)
 		(fields_autoplaced yes)
-		(property "Reference" "#PWR0205"
+		(property "Reference" "#PWR023"
 			(at 55.88 102.87 0)
 			(effects
@@
 			(project "transistor-clock"
 				(path "/ce10d5bc-995e-4952-aa76-0a08f713a0f2/2c36a9e9-de42-4705-9ad4-94f4cc168e2f/45f6b4b3-4b31-405d-8488-938c33278b8a"
-					(reference "#PWR0227")
+					(reference "#PWR038")
 					(unit 1)
 				)
 				(path "/ce10d5bc-995e-4952-aa76-0a08f713a0f2/2c36a9e9-de42-4705-9ad4-94f4cc168e2f/6e22859f-9bca-4d3f-9901-b092abdf20a9"
-					(reference "#PWR0205")
+					(reference "#PWR023")
 					(unit 1)
 				)
@@
 		(dnp no)
 		(fields_autoplaced yes)
-		(property "Reference" "#PWR010"
+		(property "Reference" "#PWR025"
 			(at 161.29 111.76 0)
 			(effects
@@
 			(project "transistor-clock"
 				(path "/ce10d5bc-995e-4952-aa76-0a08f713a0f2/2c36a9e9-de42-4705-9ad4-94f4cc168e2f/45f6b4b3-4b31-405d-8488-938c33278b8a"
-					(reference "#PWR011")
+					(reference "#PWR040")
 					(unit 1)
 				)
 				(path "/ce10d5bc-995e-4952-aa76-0a08f713a0f2/2c36a9e9-de42-4705-9ad4-94f4cc168e2f/6e22859f-9bca-4d3f-9901-b092abdf20a9"
-					(reference "#PWR010")
+					(reference "#PWR025")
 					(unit 1)
 				)
@@
 		(dnp no)
 		(fields_autoplaced yes)
-		(property "Reference" "#PWR012"
+		(property "Reference" "#PWR024"
 			(at 161.29 104.14 0)
 			(effects
@@
 			(project "transistor-clock"
 				(path "/ce10d5bc-995e-4952-aa76-0a08f713a0f2/2c36a9e9-de42-4705-9ad4-94f4cc168e2f/45f6b4b3-4b31-405d-8488-938c33278b8a"
-					(reference "#PWR013")
+					(reference "#PWR039")
 					(unit 1)
 				)
 				(path "/ce10d5bc-995e-4952-aa76-0a08f713a0f2/2c36a9e9-de42-4705-9ad4-94f4cc168e2f/6e22859f-9bca-4d3f-9901-b092abdf20a9"
-					(reference "#PWR012")
+					(reference "#PWR024")
 					(unit 1)
 				)
@@
 	)
 	(symbol
-		(lib_name "jk-flipflops_2")
 		(lib_id "custom:jk-flipflops")
 		(at 158.75 93.98 0)
@@
 		(on_board yes)
 		(dnp no)
-		(property "Reference" "U9"
+		(property "Reference" "U11"
 			(at 166.624 97.028 0)
 			(effects
@@
 			)
 		)
-		(property "Footprint" ""
+		(property "Footprint" "custom:module_flipflop_mpcie"
 			(at 158.75 93.98 0)
 			(effects
@@
 		(pin "34"
 		)
-		(pin "35"
+		(pin "31"
 		)
 		(pin "12"
@@
 			(project "transistor-clock"
 				(path "/ce10d5bc-995e-4952-aa76-0a08f713a0f2/2c36a9e9-de42-4705-9ad4-94f4cc168e2f/45f6b4b3-4b31-405d-8488-938c33278b8a"
-					(reference "U10")
+					(reference "U12")
 					(unit 5)
 				)
 				(path "/ce10d5bc-995e-4952-aa76-0a08f713a0f2/2c36a9e9-de42-4705-9ad4-94f4cc168e2f/6e22859f-9bca-4d3f-9901-b092abdf20a9"
-					(reference "U9")
+					(reference "U11")
 					(unit 5)
 				)

Commit message: added module for PSU
Parts:
- U5: renamed from U11; value ~ -> flipflop; LCSC Part # (none) -> C185937
Changed lines of the file:
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@@
 		(dnp no)
 		(fields_autoplaced yes)
-		(property "Reference" "U11"
+		(property "Reference" "U5"
 			(at 73.2633 105.0869 0)
 			(effects
@@
 			)
 		)
-		(property "Value" "~"
+		(property "Value" "flipflop"
 			(at 66.04 105.41 0)
 			(effects
@@
 			)
 		)
-		(property "LCSC Part #" ""
+		(property "LCSC Part #" "C185937"
 			(at 66.04 105.41 0)
 			(effects
@@
 			(project "transistor-clock"
 				(path "/ce10d5bc-995e-4952-aa76-0a08f713a0f2/2c36a9e9-de42-4705-9ad4-94f4cc168e2f/45f6b4b3-4b31-405d-8488-938c33278b8a"
-					(reference "U12")
+					(reference "U6")
 					(unit 1)
 				)
 				(path "/ce10d5bc-995e-4952-aa76-0a08f713a0f2/2c36a9e9-de42-4705-9ad4-94f4cc168e2f/6e22859f-9bca-4d3f-9901-b092abdf20a9"
-					(reference "U11")
+					(reference "U5")
 					(unit 1)
 				)
@@
 		(dnp no)
 		(fields_autoplaced yes)
-		(property "Reference" "U11"
+		(property "Reference" "U5"
 			(at 99.9333 105.0869 0)
 			(effects
@@
 			)
 		)
-		(property "Value" "~"
+		(property "Value" "flipflop"
 			(at 92.71 105.41 0)
 			(effects
@@
 			)
 		)
-		(property "LCSC Part #" ""
+		(property "LCSC Part #" "C185937"
 			(at 92.71 105.41 0)
 			(effects
@@
 			(project "transistor-clock"
 				(path "/ce10d5bc-995e-4952-aa76-0a08f713a0f2/2c36a9e9-de42-4705-9ad4-94f4cc168e2f/45f6b4b3-4b31-405d-8488-938c33278b8a"
-					(reference "U12")
+					(reference "U6")
 					(unit 2)
 				)
 				(path "/ce10d5bc-995e-4952-aa76-0a08f713a0f2/2c36a9e9-de42-4705-9ad4-94f4cc168e2f/6e22859f-9bca-4d3f-9901-b092abdf20a9"
-					(reference "U11")
+					(reference "U5")
 					(unit 2)
 				)
@@
 		(dnp no)
 		(fields_autoplaced yes)
-		(property "Reference" "U11"
+		(property "Reference" "U5"
 			(at 131.6833 105.0869 0)
 			(effects
@@
 			)
 		)
-		(property "Value" "~"
+		(property "Value" "flipflop"
 			(at 124.46 105.41 0)
 			(effects
@@
 			)
 		)
-		(property "LCSC Part #" ""
+		(property "LCSC Part #" "C185937"
 			(at 124.46 105.41 0)
 			(effects
@@
 			(project "transistor-clock"
 				(path "/ce10d5bc-995e-4952-aa76-0a08f713a0f2/2c36a9e9-de42-4705-9ad4-94f4cc168e2f/45f6b4b3-4b31-405d-8488-938c33278b8a"
-					(reference "U12")
+					(reference "U6")
 					(unit 3)
 				)
 				(path "/ce10d5bc-995e-4952-aa76-0a08f713a0f2/2c36a9e9-de42-4705-9ad4-94f4cc168e2f/6e22859f-9bca-4d3f-9901-b092abdf20a9"
-					(reference "U11")
+					(reference "U5")
 					(unit 3)
 				)
@@
 		(on_board yes)
 		(dnp no)
-		(property "Reference" "U11"
+		(property "Reference" "U5"
 			(at 166.624 97.028 0)
 			(effects
@@
 			)
 		)
-		(property "Value" "~"
+		(property "Value" "flipflop"
 			(at 158.75 93.98 0)
 			(effects
@@
 			)
 		)
-		(property "LCSC Part #" ""
+		(property "LCSC Part #" "C185937"
 			(at 158.75 93.98 0)
 			(effects
@@
 			(project "transistor-clock"
 				(path "/ce10d5bc-995e-4952-aa76-0a08f713a0f2/2c36a9e9-de42-4705-9ad4-94f4cc168e2f/45f6b4b3-4b31-405d-8488-938c33278b8a"
-					(reference "U12")
+					(reference "U6")
 					(unit 5)
 				)
 				(path "/ce10d5bc-995e-4952-aa76-0a08f713a0f2/2c36a9e9-de42-4705-9ad4-94f4cc168e2f/6e22859f-9bca-4d3f-9901-b092abdf20a9"
-					(reference "U11")
+					(reference "U5")
 					(unit 5)
 				)

Commit message: flipflop sims
Connections:
- net +3V3: now also U5.26 (Pre), U5.51 (Pre), U5.8 (Pre)
- no-connect marks 3 -> 0
Changed lines of the file:
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@@
+	)
+	(junction
+		(at 71.12 99.06)
+		(diameter 0)
+		(color 0 0 0 0)
 	)
 	(junction
@@
 	)
 	(junction
+		(at 97.79 99.06)
+		(diameter 0)
+		(color 0 0 0 0)
+	)
+	(junction
 		(at 85.09 111.76)
 		(diameter 0)
@@
 	)
 	(junction
+		(at 119.38 99.06)
+		(diameter 0)
+		(color 0 0 0 0)
+	)
+	(junction
 		(at 62.23 119.38)
 		(diameter 0)
@@
 		(color 0 0 0 0)
 	)
-	(no_connect
-		(at 129.54 104.14)
-	)
-	(no_connect
-		(at 71.12 104.14)
-	)
-	(no_connect
-		(at 97.79 104.14)
-	)
 	(wire
 		(pts
@@
 	(wire
 		(pts
+			(xy 97.79 99.06) (xy 119.38 99.06)
+		)
+		(stroke
+			(width 0)
+			(type default)
+		)
+	)
+	(wire
+		(pts
 			(xy 87.63 109.22) (xy 87.63 119.38)
 		)
@@
 	(wire
 		(pts
-			(xy 87.63 99.06) (xy 119.38 99.06)
+			(xy 87.63 99.06) (xy 97.79 99.06)
 		)
 		(stroke
@@
 	(wire
 		(pts
-			(xy 55.88 99.06) (xy 87.63 99.06)
+			(xy 55.88 99.06) (xy 71.12 99.06)
 		)
 		(stroke
@@
 	(wire
 		(pts
+			(xy 71.12 99.06) (xy 87.63 99.06)
+		)
+		(stroke
+			(width 0)
+			(type default)
+		)
+	)
+	(wire
+		(pts
 			(xy 62.23 111.76) (xy 62.23 114.3)
 		)
@@
 	(wire
 		(pts
+			(xy 129.54 99.06) (xy 119.38 99.06)
+		)
+		(stroke
+			(width 0)
+			(type default)
+		)
+	)
+	(wire
+		(pts
 			(xy 87.63 99.06) (xy 87.63 109.22)
 		)
@@
 	(wire
 		(pts
+			(xy 129.54 104.14) (xy 129.54 99.06)
+		)
+		(stroke
+			(width 0)
+			(type default)
+		)
+	)
+	(wire
+		(pts
 			(xy 85.09 85.09) (xy 85.09 111.76)
 		)
@@
 	(wire
 		(pts
+			(xy 71.12 99.06) (xy 71.12 104.14)
+		)
+		(stroke
+			(width 0)
+			(type default)
+		)
+	)
+	(wire
+		(pts
 			(xy 62.23 109.22) (xy 62.23 111.76)
 		)
@@
 		)
 		(stroke
+			(width 0)
+			(type default)
+		)
+	)
+	(wire
+		(pts
+			(xy 97.79 99.06) (xy 97.79 104.14)
+		)
+		(stroke
