File: transistor-clock.kicad_sch (KiCad schematic)
At the start: 44 parts, among them J1 Screw_Terminal_01x02, J2 Conn_01x01_Socket, J3 Conn_01x01_Socket, J4 Conn_01x01_Socket, J5 Conn_01x01_Socket, J6 Conn_01x01_Socket, J7 Conn_01x01_Socket, Q1 MMBT3904, Q2 MMBT3904, Q3 MMBT3904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

Commit message: routing
Parts:
- J2, J3, J4, J5, J6, J7, TR1, TR2: now left out of the parts list
Connections:
- net VSS: now also TR2.7; no longer TR2.12
- net at Q9.2 (E): now also TR2.12; no longer TR2.7
Changed lines of the file:
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@@
 		)
 	)
-	(label "Sqr1"
+	(label "Sqr2"
 		(at 128.27 129.54 0)
 		(effects
@@
 		)
 	)
-	(label "Sqr2"
+	(label "Sqr1"
 		(at 128.27 144.78 0)
 		(effects
@@
 		(unit 1)
 		(exclude_from_sim no)
-		(in_bom yes)
+		(in_bom no)
 		(on_board yes)
 		(dnp no)
@@
 		(unit 1)
 		(exclude_from_sim no)
-		(in_bom yes)
+		(in_bom no)
 		(on_board yes)
 		(dnp no)
@@
 		(unit 1)
 		(exclude_from_sim no)
-		(in_bom yes)
+		(in_bom no)
 		(on_board yes)
 		(dnp no)
@@
 		(unit 1)
 		(exclude_from_sim no)
-		(in_bom yes)
+		(in_bom no)
 		(on_board yes)
 		(dnp no)
@@
 		(unit 1)
 		(exclude_from_sim no)
-		(in_bom yes)
+		(in_bom no)
 		(on_board yes)
 		(dnp no)
@@
 		(lib_id "Transformer:TRANSF3")
 		(at 113.03 137.16 0)
-		(mirror x)
 		(unit 1)
 		(exclude_from_sim no)
-		(in_bom yes)
+		(in_bom no)
 		(on_board yes)
 		(dnp no)
 		(property "Reference" "TR2"
-			(at 113.03 149.0515 0)
+			(at 113.03 125.2685 0)
 			(effects
 				(font
@@
 		)
 		(property "Value" "CL2-20-12"
-			(at 113.03 146.6272 0)
+			(at 113.03 127.6928 0)
 			(effects
 				(font
@@
 		(unit 1)
 		(exclude_from_sim no)
-		(in_bom yes)
+		(in_bom no)
 		(on_board yes)
 		(dnp no)
@@
 		(unit 1)
 		(exclude_from_sim no)
-		(in_bom yes)
+		(in_bom no)
 		(on_board yes)
 		(dnp no)

Commit message: flipflop wip
Parts:
- added F1, F3, F4: 250mA?, Fuse:Fuse_Littelfuse-NANO2-885, symbol Device:Fuse
- added F2: 2A?, Fuse:Fuse_Littelfuse-NANO2-885, symbol Device:Fuse
- added H1, H2, H3, H4, H5, H6: MountingHole, MountingHole:MountingHole_4.3mm_M4_DIN965, symbol Mechanical:MountingHole
Connections:
- net +3V3: now also F2.2; no longer U14.2 (VCC)
- net VDD: now also F4.2; no longer U15.2 (VCC)
- net VSS: now also F3.2; no longer U16.3 (GND)
- net AC_N: now reaches J1.1 (Pin_1), TR1.1
- net at J1.2 (Pin_2): now also F1.1; no longer TR1.4
- new net: F4.1, U15.2 (VCC)
- new net: F2.1, U14.2 (VCC)
- new net: F3.1, U16.3 (GND)
- new net AC_L: F1.2, TR1.4
Other:
- moved on the sheet: J1

Commit message: cleanup and DRC
Parts:
- added TP2: TestPoint_2Pole, Connector_PinHeader_2.54mm:PinHeader_1x02_P2.54mm_Vertical, symbol Connector:TestPoint_2Pole
Connections:
- net VSS: now also TP2.2
- net at Q9.2 (E), TR2.12: now also TP2.1
Changed lines of the file:
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@@
 	)
 	(junction
+		(at 104.14 139.7)
+		(diameter 0)
+		(color 0 0 0 0)
+	)
+	(junction
 		(at 90.17 77.47)
 		(diameter 0)
@@
 		(color 0 0 0 0)
 	)
+	(junction
+		(at 107.95 129.54)
+		(diameter 0)
+		(color 0 0 0 0)
+	)
 	(no_connect
 		(at 39.37 160.02)
@@
 	(wire
 		(pts
+			(xy 104.14 129.54) (xy 107.95 129.54)
+		)
+		(stroke
+			(width 0)
+			(type default)
+		)
+	)
+	(wire
+		(pts
 			(xy 87.63 38.1) (xy 100.33 38.1)
 		)
@@
 	(wire
 		(pts
-			(xy 88.9 139.7) (xy 107.95 139.7)
+			(xy 88.9 139.7) (xy 104.14 139.7)
 		)
 		(stroke
@@
 	(wire
 		(pts
+			(xy 104.14 139.7) (xy 107.95 139.7)
+		)
+		(stroke
+			(width 0)
+			(type default)
+		)
+	)
+	(wire
+		(pts
 			(xy 101.6 170.18) (xy 106.68 170.18)
 		)
@@
 					(unit 1)
 				)
+			)
+		)
+	)
+	(symbol
+		(lib_id "Connector:TestPoint_2Pole")
+		(at 104.14 134.62 270)
+		(unit 1)
+		(exclude_from_sim no)
+		(in_bom yes)
+		(on_board yes)
+		(dnp no)
+		(fields_autoplaced yes)
+		(property "Reference" "TP2"
+			(at 105.537 134.62 90)
+			(effects
+				(font
+					(size 1.27 1.27)
+				)
+				(justify left)
+			)
+		)
+		(property "Value" "TestPoint_2Pole"
+			(at 105.537 135.8321 90)
+			(effects
+				(font
+					(size 1.27 1.27)
+				)
+				(justify left)
+				(hide yes)
+			)
+		)
+		(property "Footprint" "Connector_PinHeader_2.54mm:PinHeader_1x02_P2.54mm_Vertical"
+			(at 104.14 134.62 0)
+			(effects
+				(font
+					(size 1.27 1.27)
+				)
+				(hide yes)
+			)
+		)
+		(property "Datasheet" "~"
+			(at 104.14 134.62 0)
+			(effects
+				(font
+					(size 1.27 1.27)
+				)
+				(hide yes)
+			)
+		)
+		(property "Description" "2-polar test point"
+			(at 104.14 134.62 0)
+			(effects
+				(font
+					(size 1.27 1.27)
+				)
+				(hide yes)
+			)
+		)
+		(pin "1"
+		)
+		(pin "2"
+		)
+		(instances
+			(project "transistor-clock"
+				(path "/ce10d5bc-995e-4952-aa76-0a08f713a0f2"
+					(reference "TP2")
+					(unit 1)
+				)

Commit message: change clock to 2hz? does input flipflop half it?
Parts:
- Q2, Q9: LCSC Part # C20526v -> C20526
- R3, R5: value 15k -> 47k; LCSC Part # C22809 -> (none)
- RV1, RV2: value 5k -> 30k; footprint Potentiometer_SMD:Potentiometer_Bourns_3214J_Horizontal -> Potentiometer_THT:Potentiometer_Bourns_3296W_Vertical; LCSC Part # C58391 -> (none)
Changed lines of the file:
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@@
 			)
 		)
-		(property "Value" "5k"
+		(property "Value" "30k"
 			(at 54.356 164.846 0)
 			(effects
@@
 			)
 		)
-		(property "Footprint" "Potentiometer_SMD:Potentiometer_Bourns_3214J_Horizontal"
+		(property "Footprint" "Potentiometer_THT:Potentiometer_Bourns_3296W_Vertical"
 			(at 63.5 163.83 0)
 			(effects
@@
 			)
 		)
-		(property "Description" "Potentiometer"
+		(property "Description" "Bourns 3296W-1-203LF"
 			(at 63.5 163.83 0)
 			(effects
@@
 			)
 		)
-		(property "LCSC Part #" "C58391"
+		(property "LCSC Part #" ""
 			(at 63.5 163.83 0)
 			(effects
@@
 			)
 		)
-		(property "Value" "5k"
+		(property "Value" "30k"
 			(at 47.244 164.592 0)
 			(effects
@@
 			)
 		)
-		(property "Footprint" "Potentiometer_SMD:Potentiometer_Bourns_3214J_Horizontal"
+		(property "Footprint" "Potentiometer_THT:Potentiometer_Bourns_3296W_Vertical"
 			(at 39.37 163.83 0)
 			(effects
@@
 			)
 		)
-		(property "Description" "Potentiometer"
+		(property "Description" "Bourns 3296W-1-203LF"
 			(at 39.37 163.83 0)
 			(effects
@@
 			)
 		)
-		(property "LCSC Part #" "C58391"
+		(property "LCSC Part #" ""
 			(at 39.37 163.83 0)
 			(effects
@@
 			)
 		)
-		(property "Value" "15k"
+		(property "Value" "47k"
 			(at 65.278 172.6621 0)
 			(effects
@@
 			)
 		)
-		(property "LCSC Part #" "C22809"
+		(property "LCSC Part #" ""
+			(at 63.5 171.45 0)
+			(effects
+				(font
+					(size 1.27 1.27)
+				)
+				(hide yes)
+			)
+		)
+		(property "Field6" ""
 			(at 63.5 171.45 0)
 			(effects
@@
 			)
 		)
-		(property "LCSC Part #" "C20526v"
+		(property "LCSC Part #" "C20526"
 			(at 35.56 133.35 0)
 			(effects
@@
 			)
 		)
-		(property "Value" "15k"
+		(property "Value" "47k"
 			(at 41.148 172.6621 0)
 			(effects
@@
 			)
 		)
-		(property "LCSC Part #" "C22809"
+		(property "LCSC Part #" ""
 			(at 39.37 171.45 0)
 			(effects
@@
 			)
 		)
-		(property "LCSC Part #" "C20526v"
+		(property "LCSC Part #" "C20526"
 			(at 105.41 121.92 0)
 			(effects
