File: modules/bin-to-dec/bin-to-dec/nand.kicad_sch (KiCad schematic)
At the start: 4 parts, among them Q100 2N7002, Q101 2N7002, Q102 DMP3099L, Q99 DMP3099L

Commit message: routed on bdc
Parts:
- renumbered Q102 to Q10, Q99 to Q7, Q100 to Q8, Q101 to Q9
Changed lines of the file:
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@@
 		(dnp no)
 		(fields_autoplaced yes)
-		(property "Reference" "#PWR040"
+		(property "Reference" "#PWR011"
 			(at 147.32 101.6 0)
 			(effects
@@
 				(path "/b244e12b-f85f-4579-ba5e-848643f54694/5653fc28-2bc8-4af2-8007-5d6d268cbb44/bb5d11ea-2665-4696-a8b1-333e14f91e52"
 					(reference "#PWR046")
+					(unit 1)
+				)
+				(path "/b244e12b-f85f-4579-ba5e-848643f54694/56916597-06d0-4a11-97bd-1503266c17ac/8ee20511-ed8c-440b-be49-5bddea04a22c"
+					(reference "#PWR011")
+					(unit 1)
+				)
+				(path "/b244e12b-f85f-4579-ba5e-848643f54694/56916597-06d0-4a11-97bd-1503266c17ac/a252f2da-4fcb-47bd-92d9-0d9a35376730"
+					(reference "#PWR017")
+					(unit 1)
+				)
+				(path "/b244e12b-f85f-4579-ba5e-848643f54694/56916597-06d0-4a11-97bd-1503266c17ac/bb5d11ea-2665-4696-a8b1-333e14f91e52"
+					(reference "#PWR057")
 					(unit 1)
 				)
@@
 		(dnp no)
 		(fields_autoplaced yes)
-		(property "Reference" "#PWR039"
+		(property "Reference" "#PWR010"
 			(at 147.32 59.69 0)
 			(effects
@@
 				(path "/b244e12b-f85f-4579-ba5e-848643f54694/5653fc28-2bc8-4af2-8007-5d6d268cbb44/bb5d11ea-2665-4696-a8b1-333e14f91e52"
 					(reference "#PWR045")
+					(unit 1)
+				)
+				(path "/b244e12b-f85f-4579-ba5e-848643f54694/56916597-06d0-4a11-97bd-1503266c17ac/8ee20511-ed8c-440b-be49-5bddea04a22c"
+					(reference "#PWR010")
+					(unit 1)
+				)
+				(path "/b244e12b-f85f-4579-ba5e-848643f54694/56916597-06d0-4a11-97bd-1503266c17ac/a252f2da-4fcb-47bd-92d9-0d9a35376730"
+					(reference "#PWR016")
+					(unit 1)
+				)
+				(path "/b244e12b-f85f-4579-ba5e-848643f54694/56916597-06d0-4a11-97bd-1503266c17ac/bb5d11ea-2665-4696-a8b1-333e14f91e52"
+					(reference "#PWR028")
 					(unit 1)
 				)
@@
 		(dnp no)
 		(fields_autoplaced yes)
-		(property "Reference" "Q101"
+		(property "Reference" "Q9"
 			(at 149.987 88.9578 0)
 			(effects
@@
 				(path "/b244e12b-f85f-4579-ba5e-848643f54694/5653fc28-2bc8-4af2-8007-5d6d268cbb44/bb5d11ea-2665-4696-a8b1-333e14f91e52"
 					(reference "Q119")
+					(unit 1)
+				)
+				(path "/b244e12b-f85f-4579-ba5e-848643f54694/56916597-06d0-4a11-97bd-1503266c17ac/8ee20511-ed8c-440b-be49-5bddea04a22c"
+					(reference "Q9")
+					(unit 1)
+				)
+				(path "/b244e12b-f85f-4579-ba5e-848643f54694/56916597-06d0-4a11-97bd-1503266c17ac/a252f2da-4fcb-47bd-92d9-0d9a35376730"
+					(reference "Q25")
+					(unit 1)
+				)
+				(path "/b244e12b-f85f-4579-ba5e-848643f54694/56916597-06d0-4a11-97bd-1503266c17ac/bb5d11ea-2665-4696-a8b1-333e14f91e52"
+					(reference "Q61")
 					(unit 1)
 				)
@@
 		(on_board yes)
 		(dnp no)
-		(property "Reference" "Q102"
+		(property "Reference" "Q10"
 			(at 157.353 62.1722 0)
 			(effects
@@
 				(path "/b244e12b-f85f-4579-ba5e-848643f54694/5653fc28-2bc8-4af2-8007-5d6d268cbb44/bb5d11ea-2665-4696-a8b1-333e14f91e52"
 					(reference "Q120")
+					(unit 1)
+				)
+				(path "/b244e12b-f85f-4579-ba5e-848643f54694/56916597-06d0-4a11-97bd-1503266c17ac/8ee20511-ed8c-440b-be49-5bddea04a22c"
+					(reference "Q10")
+					(unit 1)
+				)
+				(path "/b244e12b-f85f-4579-ba5e-848643f54694/56916597-06d0-4a11-97bd-1503266c17ac/a252f2da-4fcb-47bd-92d9-0d9a35376730"
+					(reference "Q26")
+					(unit 1)
+				)
+				(path "/b244e12b-f85f-4579-ba5e-848643f54694/56916597-06d0-4a11-97bd-1503266c17ac/bb5d11ea-2665-4696-a8b1-333e14f91e52"
+					(reference "Q62")
 					(unit 1)
 				)
@@
 		(dnp no)
 		(fields_autoplaced yes)
-		(property "Reference" "Q100"
+		(property "Reference" "Q8"
 			(at 149.987 74.9878 0)
 			(effects
@@
 				(path "/b244e12b-f85f-4579-ba5e-848643f54694/5653fc28-2bc8-4af2-8007-5d6d268cbb44/bb5d11ea-2665-4696-a8b1-333e14f91e52"
 					(reference "Q118")
+					(unit 1)
+				)
+				(path "/b244e12b-f85f-4579-ba5e-848643f54694/56916597-06d0-4a11-97bd-1503266c17ac/8ee20511-ed8c-440b-be49-5bddea04a22c"
+					(reference "Q8")
+					(unit 1)
+				)
+				(path "/b244e12b-f85f-4579-ba5e-848643f54694/56916597-06d0-4a11-97bd-1503266c17ac/a252f2da-4fcb-47bd-92d9-0d9a35376730"
+					(reference "Q24")
+					(unit 1)
+				)
+				(path "/b244e12b-f85f-4579-ba5e-848643f54694/56916597-06d0-4a11-97bd-1503266c17ac/bb5d11ea-2665-4696-a8b1-333e14f91e52"
+					(reference "Q60")
 					(unit 1)
 				)
@@
 		(on_board yes)
 		(dnp no)
-		(property "Reference" "Q99"
+		(property "Reference" "Q7"
 			(at 138.557 62.1722 0)
 			(effects
@@
 					(unit 1)
 				)
+				(path "/b244e12b-f85f-4579-ba5e-848643f54694/56916597-06d0-4a11-97bd-1503266c17ac/8ee20511-ed8c-440b-be49-5bddea04a22c"
+					(reference "Q7")
+					(unit 1)
+				)
+				(path "/b244e12b-f85f-4579-ba5e-848643f54694/56916597-06d0-4a11-97bd-1503266c17ac/a252f2da-4fcb-47bd-92d9-0d9a35376730"
+					(reference "Q23")
+					(unit 1)
+				)
+				(path "/b244e12b-f85f-4579-ba5e-848643f54694/56916597-06d0-4a11-97bd-1503266c17ac/bb5d11ea-2665-4696-a8b1-333e14f91e52"
+					(reference "Q59")
+					(unit 1)
+				)

Commit message: went from routed bin-to-dec to gate only
Parts:
- renumbered Q8 to Q10, Q9 to Q11, Q10 to Q12, Q7 to Q9
Changed lines of the file:
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@@
 		(dnp no)
 		(fields_autoplaced yes)
-		(property "Reference" "#PWR011"
+		(property "Reference" "#PWR08"
 			(at 147.32 101.6 0)
 			(effects
@@
 		(instances
 			(project "bin-to-dec"
-				(path "/b244e12b-f85f-4579-ba5e-848643f54694/5653fc28-2bc8-4af2-8007-5d6d268cbb44/8ee20511-ed8c-440b-be49-5bddea04a22c"
-					(reference "#PWR052")
-					(unit 1)
-				)
-				(path "/b244e12b-f85f-4579-ba5e-848643f54694/5653fc28-2bc8-4af2-8007-5d6d268cbb44/a252f2da-4fcb-47bd-92d9-0d9a35376730"
-					(reference "#PWR040")
-					(unit 1)
-				)
-				(path "/b244e12b-f85f-4579-ba5e-848643f54694/5653fc28-2bc8-4af2-8007-5d6d268cbb44/bb5d11ea-2665-4696-a8b1-333e14f91e52"
-					(reference "#PWR046")
-					(unit 1)
-				)
-				(path "/b244e12b-f85f-4579-ba5e-848643f54694/56916597-06d0-4a11-97bd-1503266c17ac/8ee20511-ed8c-440b-be49-5bddea04a22c"
-					(reference "#PWR011")
-					(unit 1)
-				)
-				(path "/b244e12b-f85f-4579-ba5e-848643f54694/56916597-06d0-4a11-97bd-1503266c17ac/a252f2da-4fcb-47bd-92d9-0d9a35376730"
-					(reference "#PWR017")
-					(unit 1)
-				)
-				(path "/b244e12b-f85f-4579-ba5e-848643f54694/56916597-06d0-4a11-97bd-1503266c17ac/bb5d11ea-2665-4696-a8b1-333e14f91e52"
-					(reference "#PWR057")
+				(path "/b244e12b-f85f-4579-ba5e-848643f54694/8559444b-ed80-4591-94fd-530ce32ce577"
+					(reference "#PWR026")
+					(unit 1)
+				)
+				(path "/b244e12b-f85f-4579-ba5e-848643f54694/9ee95dfd-f3ee-48c6-9665-30ae2b1f5b54"
+					(reference "#PWR016")
+					(unit 1)
+				)
+				(path "/b244e12b-f85f-4579-ba5e-848643f54694/c84f6135-6667-4c7e-9ce8-5338f93253d6"
+					(reference "#PWR08")
 					(unit 1)
 				)
@@
 		(dnp no)
 		(fields_autoplaced yes)
-		(property "Reference" "#PWR010"
+		(property "Reference" "#PWR07"
 			(at 147.32 59.69 0)
 			(effects
@@
 		(instances
 			(project "bin-to-dec"
-				(path "/b244e12b-f85f-4579-ba5e-848643f54694/5653fc28-2bc8-4af2-8007-5d6d268cbb44/8ee20511-ed8c-440b-be49-5bddea04a22c"
-					(reference "#PWR051")
-					(unit 1)
-				)
-				(path "/b244e12b-f85f-4579-ba5e-848643f54694/5653fc28-2bc8-4af2-8007-5d6d268cbb44/a252f2da-4fcb-47bd-92d9-0d9a35376730"
-					(reference "#PWR039")
-					(unit 1)
-				)
-				(path "/b244e12b-f85f-4579-ba5e-848643f54694/5653fc28-2bc8-4af2-8007-5d6d268cbb44/bb5d11ea-2665-4696-a8b1-333e14f91e52"
-					(reference "#PWR045")
-					(unit 1)
-				)
-				(path "/b244e12b-f85f-4579-ba5e-848643f54694/56916597-06d0-4a11-97bd-1503266c17ac/8ee20511-ed8c-440b-be49-5bddea04a22c"
-					(reference "#PWR010")
-					(unit 1)
-				)
-				(path "/b244e12b-f85f-4579-ba5e-848643f54694/56916597-06d0-4a11-97bd-1503266c17ac/a252f2da-4fcb-47bd-92d9-0d9a35376730"
-					(reference "#PWR016")
-					(unit 1)
-				)
-				(path "/b244e12b-f85f-4579-ba5e-848643f54694/56916597-06d0-4a11-97bd-1503266c17ac/bb5d11ea-2665-4696-a8b1-333e14f91e52"
-					(reference "#PWR028")
+				(path "/b244e12b-f85f-4579-ba5e-848643f54694/8559444b-ed80-4591-94fd-530ce32ce577"
+					(reference "#PWR025")
+					(unit 1)
+				)
+				(path "/b244e12b-f85f-4579-ba5e-848643f54694/9ee95dfd-f3ee-48c6-9665-30ae2b1f5b54"
+					(reference "#PWR015")
+					(unit 1)
+				)
+				(path "/b244e12b-f85f-4579-ba5e-848643f54694/c84f6135-6667-4c7e-9ce8-5338f93253d6"
+					(reference "#PWR07")
 					(unit 1)
 				)
@@
 		(dnp no)
 		(fields_autoplaced yes)
-		(property "Reference" "Q9"
+		(property "Reference" "Q11"
 			(at 149.987 88.9578 0)
 			(effects
@@
 		(instances
 			(project "bin-to-dec"
-				(path "/b244e12b-f85f-4579-ba5e-848643f54694/5653fc28-2bc8-4af2-8007-5d6d268cbb44/8ee20511-ed8c-440b-be49-5bddea04a22c"
-					(reference "Q135")
-					(unit 1)
-				)
-				(path "/b244e12b-f85f-4579-ba5e-848643f54694/5653fc28-2bc8-4af2-8007-5d6d268cbb44/a252f2da-4fcb-47bd-92d9-0d9a35376730"
-					(reference "Q101")
-					(unit 1)
-				)
-				(path "/b244e12b-f85f-4579-ba5e-848643f54694/5653fc28-2bc8-4af2-8007-5d6d268cbb44/bb5d11ea-2665-4696-a8b1-333e14f91e52"
-					(reference "Q119")
-					(unit 1)
-				)
-				(path "/b244e12b-f85f-4579-ba5e-848643f54694/56916597-06d0-4a11-97bd-1503266c17ac/8ee20511-ed8c-440b-be49-5bddea04a22c"
-					(reference "Q9")
-					(unit 1)
-				)
-				(path "/b244e12b-f85f-4579-ba5e-848643f54694/56916597-06d0-4a11-97bd-1503266c17ac/a252f2da-4fcb-47bd-92d9-0d9a35376730"
-					(reference "Q25")
-					(unit 1)
-				)
-				(path "/b244e12b-f85f-4579-ba5e-848643f54694/56916597-06d0-4a11-97bd-1503266c17ac/bb5d11ea-2665-4696-a8b1-333e14f91e52"
+				(path "/b244e12b-f85f-4579-ba5e-848643f54694/8559444b-ed80-4591-94fd-530ce32ce577"
 					(reference "Q61")
+					(unit 1)
+				)
+				(path "/b244e12b-f85f-4579-ba5e-848643f54694/9ee95dfd-f3ee-48c6-9665-30ae2b1f5b54"
+					(reference "Q33")
+					(unit 1)
+				)
+				(path "/b244e12b-f85f-4579-ba5e-848643f54694/c84f6135-6667-4c7e-9ce8-5338f93253d6"
+					(reference "Q11")
 					(unit 1)
 				)
@@
 		(on_board yes)
 		(dnp no)
-		(property "Reference" "Q10"
+		(property "Reference" "Q12"
 			(at 157.353 62.1722 0)
 			(effects
@@
 		(instances
 			(project "bin-to-dec"
-				(path "/b244e12b-f85f-4579-ba5e-848643f54694/5653fc28-2bc8-4af2-8007-5d6d268cbb44/8ee20511-ed8c-440b-be49-5bddea04a22c"
-					(reference "Q136")
-					(unit 1)
-				)
-				(path "/b244e12b-f85f-4579-ba5e-848643f54694/5653fc28-2bc8-4af2-8007-5d6d268cbb44/a252f2da-4fcb-47bd-92d9-0d9a35376730"
-					(reference "Q102")
-					(unit 1)
-				)
-				(path "/b244e12b-f85f-4579-ba5e-848643f54694/5653fc28-2bc8-4af2-8007-5d6d268cbb44/bb5d11ea-2665-4696-a8b1-333e14f91e52"
-					(reference "Q120")
-					(unit 1)
-				)
-				(path "/b244e12b-f85f-4579-ba5e-848643f54694/56916597-06d0-4a11-97bd-1503266c17ac/8ee20511-ed8c-440b-be49-5bddea04a22c"
-					(reference "Q10")
-					(unit 1)
-				)
-				(path "/b244e12b-f85f-4579-ba5e-848643f54694/56916597-06d0-4a11-97bd-1503266c17ac/a252f2da-4fcb-47bd-92d9-0d9a35376730"
-					(reference "Q26")
-					(unit 1)
-				)
-				(path "/b244e12b-f85f-4579-ba5e-848643f54694/56916597-06d0-4a11-97bd-1503266c17ac/bb5d11ea-2665-4696-a8b1-333e14f91e52"
+				(path "/b244e12b-f85f-4579-ba5e-848643f54694/8559444b-ed80-4591-94fd-530ce32ce577"
 					(reference "Q62")
+					(unit 1)
+				)
+				(path "/b244e12b-f85f-4579-ba5e-848643f54694/9ee95dfd-f3ee-48c6-9665-30ae2b1f5b54"
+					(reference "Q34")
+					(unit 1)
+				)
+				(path "/b244e12b-f85f-4579-ba5e-848643f54694/c84f6135-6667-4c7e-9ce8-5338f93253d6"
+					(reference "Q12")
 					(unit 1)
 				)
@@
 		(dnp no)
 		(fields_autoplaced yes)
-		(property "Reference" "Q8"
+		(property "Reference" "Q10"
 			(at 149.987 74.9878 0)
 			(effects
@@
 		(instances
 			(project "bin-to-dec"
-				(path "/b244e12b-f85f-4579-ba5e-848643f54694/5653fc28-2bc8-4af2-8007-5d6d268cbb44/8ee20511-ed8c-440b-be49-5bddea04a22c"
-					(reference "Q134")
-					(unit 1)
-				)
-				(path "/b244e12b-f85f-4579-ba5e-848643f54694/5653fc28-2bc8-4af2-8007-5d6d268cbb44/a252f2da-4fcb-47bd-92d9-0d9a35376730"
-					(reference "Q100")
-					(unit 1)
-				)
-				(path "/b244e12b-f85f-4579-ba5e-848643f54694/5653fc28-2bc8-4af2-8007-5d6d268cbb44/bb5d11ea-2665-4696-a8b1-333e14f91e52"
-					(reference "Q118")
-					(unit 1)
-				)
-				(path "/b244e12b-f85f-4579-ba5e-848643f54694/56916597-06d0-4a11-97bd-1503266c17ac/8ee20511-ed8c-440b-be49-5bddea04a22c"
-					(reference "Q8")
-					(unit 1)
-				)
-				(path "/b244e12b-f85f-4579-ba5e-848643f54694/56916597-06d0-4a11-97bd-1503266c17ac/a252f2da-4fcb-47bd-92d9-0d9a35376730"
-					(reference "Q24")
-					(unit 1)
-				)
-				(path "/b244e12b-f85f-4579-ba5e-848643f54694/56916597-06d0-4a11-97bd-1503266c17ac/bb5d11ea-2665-4696-a8b1-333e14f91e52"
+				(path "/b244e12b-f85f-4579-ba5e-848643f54694/8559444b-ed80-4591-94fd-530ce32ce577"
 					(reference "Q60")
+					(unit 1)
+				)
+				(path "/b244e12b-f85f-4579-ba5e-848643f54694/9ee95dfd-f3ee-48c6-9665-30ae2b1f5b54"
+					(reference "Q32")
+					(unit 1)
+				)
+				(path "/b244e12b-f85f-4579-ba5e-848643f54694/c84f6135-6667-4c7e-9ce8-5338f93253d6"
+					(reference "Q10")
 					(unit 1)
 				)
@@
 		(on_board yes)
 		(dnp no)
-		(property "Reference" "Q7"
+		(property "Reference" "Q9"
 			(at 138.557 62.1722 0)
 			(effects
@@
 		(instances
 			(project "bin-to-dec"
-				(path "/b244e12b-f85f-4579-ba5e-848643f54694/5653fc28-2bc8-4af2-8007-5d6d268cbb44/8ee20511-ed8c-440b-be49-5bddea04a22c"
-					(reference "Q133")
-					(unit 1)
-				)
-				(path "/b244e12b-f85f-4579-ba5e-848643f54694/5653fc28-2bc8-4af2-8007-5d6d268cbb44/a252f2da-4fcb-47bd-92d9-0d9a35376730"
-					(reference "Q99")
-					(unit 1)
-				)
-				(path "/b244e12b-f85f-4579-ba5e-848643f54694/5653fc28-2bc8-4af2-8007-5d6d268cbb44/bb5d11ea-2665-4696-a8b1-333e14f91e52"
-					(reference "Q117")
-					(unit 1)
-				)
-				(path "/b244e12b-f85f-4579-ba5e-848643f54694/56916597-06d0-4a11-97bd-1503266c17ac/8ee20511-ed8c-440b-be49-5bddea04a22c"
-					(reference "Q7")
-					(unit 1)
-				)
-				(path "/b244e12b-f85f-4579-ba5e-848643f54694/56916597-06d0-4a11-97bd-1503266c17ac/a252f2da-4fcb-47bd-92d9-0d9a35376730"
-					(reference "Q23")
-					(unit 1)
-				)
-				(path "/b244e12b-f85f-4579-ba5e-848643f54694/56916597-06d0-4a11-97bd-1503266c17ac/bb5d11ea-2665-4696-a8b1-333e14f91e52"
+				(path "/b244e12b-f85f-4579-ba5e-848643f54694/8559444b-ed80-4591-94fd-530ce32ce577"
 					(reference "Q59")
 					(unit 1)
 				)
+				(path "/b244e12b-f85f-4579-ba5e-848643f54694/9ee95dfd-f3ee-48c6-9665-30ae2b1f5b54"
+					(reference "Q31")
+					(unit 1)
+				)
+				(path "/b244e12b-f85f-4579-ba5e-848643f54694/c84f6135-6667-4c7e-9ce8-5338f93253d6"
+					(reference "Q9")
+					(unit 1)
+				)
