File: modules/bin-to-dec/bin-to-dec/nand4.kicad_sch (KiCad schematic)
At the start: 8 parts, among them Q109 DMP3099L, Q110 DMP3099L, Q111 2N7002, Q112 2N7002, Q113 2N7002, Q114 2N7002, Q115 DMP3099L, Q116 DMP3099L

Commit message: routed on bdc
Parts:
- renumbered Q109 to Q39, Q110 to Q40, Q111 to Q41, Q112 to Q42, Q113 to Q43, Q114 to Q44, Q115 to Q45, Q116 to Q46
Changed lines of the file:
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@@
 		(dnp no)
 		(fields_autoplaced yes)
-		(property "Reference" "Q114"
+		(property "Reference" "Q44"
 			(at 147.447 124.5178 0)
 			(effects
@@
 					(unit 1)
 				)
+				(path "/b244e12b-f85f-4579-ba5e-848643f54694/56916597-06d0-4a11-97bd-1503266c17ac/f6ccbfec-8dc5-4010-ac3f-a448bba123af"
+					(reference "Q44")
+					(unit 1)
+				)
 			)
 		)
@@
 		(dnp no)
 		(fields_autoplaced yes)
-		(property "Reference" "Q111"
+		(property "Reference" "Q41"
 			(at 147.447 86.4178 0)
 			(effects
@@
 					(unit 1)
 				)
+				(path "/b244e12b-f85f-4579-ba5e-848643f54694/56916597-06d0-4a11-97bd-1503266c17ac/f6ccbfec-8dc5-4010-ac3f-a448bba123af"
+					(reference "Q41")
+					(unit 1)
+				)
 			)
 		)
@@
 		(on_board yes)
 		(dnp no)
-		(property "Reference" "Q110"
+		(property "Reference" "Q40"
 			(at 129.413 73.6022 0)
 			(effects
@@
 					(unit 1)
 				)
+				(path "/b244e12b-f85f-4579-ba5e-848643f54694/56916597-06d0-4a11-97bd-1503266c17ac/f6ccbfec-8dc5-4010-ac3f-a448bba123af"
+					(reference "Q40")
+					(unit 1)
+				)
 			)
 		)
@@
 		(on_board yes)
 		(dnp no)
-		(property "Reference" "Q116"
+		(property "Reference" "Q46"
 			(at 177.673 73.6022 0)
 			(effects
@@
 					(unit 1)
 				)
+				(path "/b244e12b-f85f-4579-ba5e-848643f54694/56916597-06d0-4a11-97bd-1503266c17ac/f6ccbfec-8dc5-4010-ac3f-a448bba123af"
+					(reference "Q46")
+					(unit 1)
+				)
 			)
 		)
@@
 		(dnp no)
 		(fields_autoplaced yes)
-		(property "Reference" "#PWR043"
+		(property "Reference" "#PWR022"
 			(at 144.78 71.12 0)
 			(effects
@@
 				(path "/b244e12b-f85f-4579-ba5e-848643f54694/5653fc28-2bc8-4af2-8007-5d6d268cbb44/f6ccbfec-8dc5-4010-ac3f-a448bba123af"
 					(reference "#PWR043")
+					(unit 1)
+				)
+				(path "/b244e12b-f85f-4579-ba5e-848643f54694/56916597-06d0-4a11-97bd-1503266c17ac/f6ccbfec-8dc5-4010-ac3f-a448bba123af"
+					(reference "#PWR022")
 					(unit 1)
 				)
@@
 		(on_board yes)
 		(dnp no)
-		(property "Reference" "Q109"
+		(property "Reference" "Q39"
 			(at 110.617 73.6022 0)
 			(effects
@@
 					(unit 1)
 				)
+				(path "/b244e12b-f85f-4579-ba5e-848643f54694/56916597-06d0-4a11-97bd-1503266c17ac/f6ccbfec-8dc5-4010-ac3f-a448bba123af"
+					(reference "Q39")
+					(unit 1)
+				)
 			)
 		)
@@
 		(on_board yes)
 		(dnp no)
-		(property "Reference" "Q115"
+		(property "Reference" "Q45"
 			(at 153.543 73.6022 0)
 			(effects
@@
 					(unit 1)
 				)
+				(path "/b244e12b-f85f-4579-ba5e-848643f54694/56916597-06d0-4a11-97bd-1503266c17ac/f6ccbfec-8dc5-4010-ac3f-a448bba123af"
+					(reference "Q45")
+					(unit 1)
+				)
 			)
 		)
@@
 		(dnp no)
 		(fields_autoplaced yes)
-		(property "Reference" "#PWR044"
+		(property "Reference" "#PWR023"
 			(at 144.78 137.16 0)
 			(effects
@@
 					(unit 1)
 				)
+				(path "/b244e12b-f85f-4579-ba5e-848643f54694/56916597-06d0-4a11-97bd-1503266c17ac/f6ccbfec-8dc5-4010-ac3f-a448bba123af"
+					(reference "#PWR023")
+					(unit 1)
+				)
 			)
 		)
@@
 		(dnp no)
 		(fields_autoplaced yes)
-		(property "Reference" "Q112"
+		(property "Reference" "Q42"
 			(at 147.447 100.3878 0)
 			(effects
@@
 					(unit 1)
 				)
+				(path "/b244e12b-f85f-4579-ba5e-848643f54694/56916597-06d0-4a11-97bd-1503266c17ac/f6ccbfec-8dc5-4010-ac3f-a448bba123af"
+					(reference "Q42")
+					(unit 1)
+				)
 			)
 		)
@@
 		(dnp no)
 		(fields_autoplaced yes)
-		(property "Reference" "Q113"
+		(property "Reference" "Q43"
 			(at 147.447 110.5478 0)
 			(effects
@@
 					(unit 1)
 				)
+				(path "/b244e12b-f85f-4579-ba5e-848643f54694/56916597-06d0-4a11-97bd-1503266c17ac/f6ccbfec-8dc5-4010-ac3f-a448bba123af"
+					(reference "Q43")
+					(unit 1)
+				)

Commit message: went from routed bin-to-dec to gate only
Parts:
- renumbered Q39 to Q1, Q40 to Q2, Q41 to Q3, Q42 to Q4, Q43 to Q5, Q44 to Q6, Q45 to Q7, Q46 to Q8
Changed lines of the file:
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@@
 		(dnp no)
 		(fields_autoplaced yes)
-		(property "Reference" "Q44"
+		(property "Reference" "Q6"
 			(at 147.447 124.5178 0)
 			(effects
@@
 		(instances
 			(project "bin-to-dec"
-				(path "/b244e12b-f85f-4579-ba5e-848643f54694/5653fc28-2bc8-4af2-8007-5d6d268cbb44/f6ccbfec-8dc5-4010-ac3f-a448bba123af"
-					(reference "Q114")
-					(unit 1)
-				)
-				(path "/b244e12b-f85f-4579-ba5e-848643f54694/56916597-06d0-4a11-97bd-1503266c17ac/f6ccbfec-8dc5-4010-ac3f-a448bba123af"
-					(reference "Q44")
+				(path "/b244e12b-f85f-4579-ba5e-848643f54694/0df26d3b-1463-4745-9b60-c38ec60dc515"
+					(reference "Q6")
 					(unit 1)
 				)
@@
 		(dnp no)
 		(fields_autoplaced yes)
-		(property "Reference" "Q41"
+		(property "Reference" "Q3"
 			(at 147.447 86.4178 0)
 			(effects
@@
 		(instances
 			(project "bin-to-dec"
-				(path "/b244e12b-f85f-4579-ba5e-848643f54694/5653fc28-2bc8-4af2-8007-5d6d268cbb44/f6ccbfec-8dc5-4010-ac3f-a448bba123af"
-					(reference "Q111")
-					(unit 1)
-				)
-				(path "/b244e12b-f85f-4579-ba5e-848643f54694/56916597-06d0-4a11-97bd-1503266c17ac/f6ccbfec-8dc5-4010-ac3f-a448bba123af"
-					(reference "Q41")
+				(path "/b244e12b-f85f-4579-ba5e-848643f54694/0df26d3b-1463-4745-9b60-c38ec60dc515"
+					(reference "Q3")
 					(unit 1)
 				)
@@
 		(on_board yes)
 		(dnp no)
-		(property "Reference" "Q40"
+		(property "Reference" "Q2"
 			(at 129.413 73.6022 0)
 			(effects
@@
 		(instances
 			(project "bin-to-dec"
-				(path "/b244e12b-f85f-4579-ba5e-848643f54694/5653fc28-2bc8-4af2-8007-5d6d268cbb44/f6ccbfec-8dc5-4010-ac3f-a448bba123af"
-					(reference "Q110")
-					(unit 1)
-				)
-				(path "/b244e12b-f85f-4579-ba5e-848643f54694/56916597-06d0-4a11-97bd-1503266c17ac/f6ccbfec-8dc5-4010-ac3f-a448bba123af"
-					(reference "Q40")
+				(path "/b244e12b-f85f-4579-ba5e-848643f54694/0df26d3b-1463-4745-9b60-c38ec60dc515"
+					(reference "Q2")
 					(unit 1)
 				)
@@
 		(on_board yes)
 		(dnp no)
-		(property "Reference" "Q46"
+		(property "Reference" "Q8"
 			(at 177.673 73.6022 0)
 			(effects
@@
 		(instances
 			(project "bin-to-dec"
-				(path "/b244e12b-f85f-4579-ba5e-848643f54694/5653fc28-2bc8-4af2-8007-5d6d268cbb44/f6ccbfec-8dc5-4010-ac3f-a448bba123af"
-					(reference "Q116")
-					(unit 1)
-				)
-				(path "/b244e12b-f85f-4579-ba5e-848643f54694/56916597-06d0-4a11-97bd-1503266c17ac/f6ccbfec-8dc5-4010-ac3f-a448bba123af"
-					(reference "Q46")
+				(path "/b244e12b-f85f-4579-ba5e-848643f54694/0df26d3b-1463-4745-9b60-c38ec60dc515"
+					(reference "Q8")
 					(unit 1)
 				)
@@
 		(dnp no)
 		(fields_autoplaced yes)
-		(property "Reference" "#PWR022"
+		(property "Reference" "#PWR05"
 			(at 144.78 71.12 0)
 			(effects
@@
 		(instances
 			(project "bin-to-dec"
-				(path "/b244e12b-f85f-4579-ba5e-848643f54694/5653fc28-2bc8-4af2-8007-5d6d268cbb44/f6ccbfec-8dc5-4010-ac3f-a448bba123af"
-					(reference "#PWR043")
-					(unit 1)
-				)
-				(path "/b244e12b-f85f-4579-ba5e-848643f54694/56916597-06d0-4a11-97bd-1503266c17ac/f6ccbfec-8dc5-4010-ac3f-a448bba123af"
-					(reference "#PWR022")
+				(path "/b244e12b-f85f-4579-ba5e-848643f54694/0df26d3b-1463-4745-9b60-c38ec60dc515"
+					(reference "#PWR05")
 					(unit 1)
 				)
@@
 		(on_board yes)
 		(dnp no)
-		(property "Reference" "Q39"
+		(property "Reference" "Q1"
 			(at 110.617 73.6022 0)
 			(effects
@@
 		(instances
 			(project "bin-to-dec"
-				(path "/b244e12b-f85f-4579-ba5e-848643f54694/5653fc28-2bc8-4af2-8007-5d6d268cbb44/f6ccbfec-8dc5-4010-ac3f-a448bba123af"
-					(reference "Q109")
-					(unit 1)
-				)
-				(path "/b244e12b-f85f-4579-ba5e-848643f54694/56916597-06d0-4a11-97bd-1503266c17ac/f6ccbfec-8dc5-4010-ac3f-a448bba123af"
-					(reference "Q39")
+				(path "/b244e12b-f85f-4579-ba5e-848643f54694/0df26d3b-1463-4745-9b60-c38ec60dc515"
+					(reference "Q1")
 					(unit 1)
 				)
@@
 		(on_board yes)
 		(dnp no)
-		(property "Reference" "Q45"
+		(property "Reference" "Q7"
 			(at 153.543 73.6022 0)
 			(effects
@@
 		(instances
 			(project "bin-to-dec"
-				(path "/b244e12b-f85f-4579-ba5e-848643f54694/5653fc28-2bc8-4af2-8007-5d6d268cbb44/f6ccbfec-8dc5-4010-ac3f-a448bba123af"
-					(reference "Q115")
-					(unit 1)
-				)
-				(path "/b244e12b-f85f-4579-ba5e-848643f54694/56916597-06d0-4a11-97bd-1503266c17ac/f6ccbfec-8dc5-4010-ac3f-a448bba123af"
-					(reference "Q45")
+				(path "/b244e12b-f85f-4579-ba5e-848643f54694/0df26d3b-1463-4745-9b60-c38ec60dc515"
+					(reference "Q7")
 					(unit 1)
 				)
@@
 		(dnp no)
 		(fields_autoplaced yes)
-		(property "Reference" "#PWR023"
+		(property "Reference" "#PWR06"
 			(at 144.78 137.16 0)
 			(effects
@@
 		(instances
 			(project "bin-to-dec"
-				(path "/b244e12b-f85f-4579-ba5e-848643f54694/5653fc28-2bc8-4af2-8007-5d6d268cbb44/f6ccbfec-8dc5-4010-ac3f-a448bba123af"
-					(reference "#PWR044")
-					(unit 1)
-				)
-				(path "/b244e12b-f85f-4579-ba5e-848643f54694/56916597-06d0-4a11-97bd-1503266c17ac/f6ccbfec-8dc5-4010-ac3f-a448bba123af"
-					(reference "#PWR023")
+				(path "/b244e12b-f85f-4579-ba5e-848643f54694/0df26d3b-1463-4745-9b60-c38ec60dc515"
+					(reference "#PWR06")
 					(unit 1)
 				)
@@
 		(dnp no)
 		(fields_autoplaced yes)
-		(property "Reference" "Q42"
+		(property "Reference" "Q4"
 			(at 147.447 100.3878 0)
 			(effects
@@
 		(instances
 			(project "bin-to-dec"
-				(path "/b244e12b-f85f-4579-ba5e-848643f54694/5653fc28-2bc8-4af2-8007-5d6d268cbb44/f6ccbfec-8dc5-4010-ac3f-a448bba123af"
-					(reference "Q112")
-					(unit 1)
-				)
-				(path "/b244e12b-f85f-4579-ba5e-848643f54694/56916597-06d0-4a11-97bd-1503266c17ac/f6ccbfec-8dc5-4010-ac3f-a448bba123af"
-					(reference "Q42")
+				(path "/b244e12b-f85f-4579-ba5e-848643f54694/0df26d3b-1463-4745-9b60-c38ec60dc515"
+					(reference "Q4")
 					(unit 1)
 				)
@@
 		(dnp no)
 		(fields_autoplaced yes)
-		(property "Reference" "Q43"
+		(property "Reference" "Q5"
 			(at 147.447 110.5478 0)
 			(effects
@@
 		(instances
 			(project "bin-to-dec"
-				(path "/b244e12b-f85f-4579-ba5e-848643f54694/5653fc28-2bc8-4af2-8007-5d6d268cbb44/f6ccbfec-8dc5-4010-ac3f-a448bba123af"
-					(reference "Q113")
-					(unit 1)
-				)
-				(path "/b244e12b-f85f-4579-ba5e-848643f54694/56916597-06d0-4a11-97bd-1503266c17ac/f6ccbfec-8dc5-4010-ac3f-a448bba123af"
-					(reference "Q43")
-					(unit 1)
-				)
+				(path "/b244e12b-f85f-4579-ba5e-848643f54694/0df26d3b-1463-4745-9b60-c38ec60dc515"
+					(reference "Q5")
+					(unit 1)
+				)
