File: modules/jkflipkflop/flipflop.kicad_sch (KiCad schematic)
At the start: 1 part

Commit message: flipflop fab output
Parts:
- C1: LCSC Part # (none) -> C14663
Changed lines of the file:
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@@
-					(unit 1)
-				)
-				(path "/8013391e-c8e7-41ee-accd-360f92f3a5d7/4285c540-e4c4-411b-82fc-69e49e6e15db"
-					(reference "#PWR030")
 					(unit 1)
 				)
 				(path "/8013391e-c8e7-41ee-accd-360f92f3a5d7/6979d884-3104-4d4d-a14e-0e449b6f5d88"
 					(reference "#PWR010")
-					(unit 1)
-				)
-				(path "/8013391e-c8e7-41ee-accd-360f92f3a5d7/6f09ade3-0ab2-4fe3-adfa-ab244f537d84"
-					(reference "#PWR061")
 					(unit 1)
 				)
@@
 			)
 		)
+		(property "LCSC Part #" "C14663"
+			(at 160.02 83.82 0)
+			(effects
+				(font
+					(size 1.27 1.27)
+				)
+				(hide yes)
+			)
+		)
 		(pin "2"
 		)
@@
 			(project "jkflipkflop"
 				(path "/8013391e-c8e7-41ee-accd-360f92f3a5d7/259d22b3-bbdc-4d1c-a30b-6746a4fa5b6c"
-					(reference "C5")
-					(unit 1)
-				)
-				(path "/8013391e-c8e7-41ee-accd-360f92f3a5d7/4285c540-e4c4-411b-82fc-69e49e6e15db"
+					(reference "C2")
+					(unit 1)
+				)
+				(path "/8013391e-c8e7-41ee-accd-360f92f3a5d7/6979d884-3104-4d4d-a14e-0e449b6f5d88"
+					(reference "C1")
+					(unit 1)
+				)
+				(path "/8013391e-c8e7-41ee-accd-360f92f3a5d7/9318a685-33db-476b-a8fe-85a58a155206"
 					(reference "C3")
-					(unit 1)
-				)
-				(path "/8013391e-c8e7-41ee-accd-360f92f3a5d7/6979d884-3104-4d4d-a14e-0e449b6f5d88"
-					(reference "C1")
-					(unit 1)
-				)
-				(path "/8013391e-c8e7-41ee-accd-360f92f3a5d7/6f09ade3-0ab2-4fe3-adfa-ab244f537d84"
-					(reference "C6")
-					(unit 1)
-				)
-				(path "/8013391e-c8e7-41ee-accd-360f92f3a5d7/9318a685-33db-476b-a8fe-85a58a155206"
-					(reference "C2")
 					(unit 1)
 				)
@@
 					(unit 1)
 				)
-				(path "/8013391e-c8e7-41ee-accd-360f92f3a5d7/4285c540-e4c4-411b-82fc-69e49e6e15db"
-					(reference "#PWR029")
-					(unit 1)
-				)
 				(path "/8013391e-c8e7-41ee-accd-360f92f3a5d7/6979d884-3104-4d4d-a14e-0e449b6f5d88"
 					(reference "#PWR09")
-					(unit 1)
-				)
-				(path "/8013391e-c8e7-41ee-accd-360f92f3a5d7/6f09ade3-0ab2-4fe3-adfa-ab244f537d84"
-					(reference "#PWR060")
 					(unit 1)
 				)
@@
 					(page "16")
 				)
-				(path "/8013391e-c8e7-41ee-accd-360f92f3a5d7/6f09ade3-0ab2-4fe3-adfa-ab244f537d84"
-					(page "26")
-				)
 			)
 		)
@@
 					(page "15")
 				)
-				(path "/8013391e-c8e7-41ee-accd-360f92f3a5d7/6f09ade3-0ab2-4fe3-adfa-ab244f537d84"
-					(page "25")
-				)
 			)
 		)
@@
 					(page "22")
 				)
-				(path "/8013391e-c8e7-41ee-accd-360f92f3a5d7/6f09ade3-0ab2-4fe3-adfa-ab244f537d84"
-					(page "27")
-				)
 			)
 		)
@@
 					(page "14")
 				)
-				(path "/8013391e-c8e7-41ee-accd-360f92f3a5d7/6f09ade3-0ab2-4fe3-adfa-ab244f537d84"
-					(page "24")
-				)
-			)
+			)
