File: modules/SSR/ssr.kicad_sch (KiCad schematic)
At the start: 2 parts

Commit message: production output for SSR module
Parts:
- R1: value R -> 330; LCSC Part # (none) -> C23138
- U1: value ~ -> GAQY210S; LCSC Part # (none) -> C7435113
Changed lines of the file:
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@@
 			)
 		)
-		(property "Value" "~"
+		(property "Value" "GAQY210S"
 			(at 133.35 115.1198 0)
 			(effects
@@
 			)
 		)
+		(property "LCSC Part #" "C7435113"
+			(at 129.54 115.57 0)
+			(effects
+				(font
+					(size 1.27 1.27)
+				)
+				(hide yes)
+			)
+		)
 		(pin "1"
 		)
@@
 		)
 		(instances
-			(project ""
+			(project "SSR"
 				(path "/e87a2758-91f7-4ecb-a75d-85b6b7264f27/0f4e9512-9bf4-4bde-8f90-172f78a48656"
 					(reference "U3")
@@
 			)
 		)
-		(property "Value" "R"
+		(property "Value" "330"
 			(at 120.7079 119.888 0)
 			(effects
@@
 			)
 		)
+		(property "LCSC Part #" "C23138"
+			(at 121.92 118.11 0)
+			(effects
+				(font
+					(size 1.27 1.27)
+				)
+				(hide yes)
+			)
+		)
 		(pin "2"
 		)
@@
 		)
 		(instances
-			(project ""
+			(project "SSR"
 				(path "/e87a2758-91f7-4ecb-a75d-85b6b7264f27/0f4e9512-9bf4-4bde-8f90-172f78a48656"
 					(reference "R3")
@@
 		)
 		(instances
-			(project ""
+			(project "SSR"
 				(path "/e87a2758-91f7-4ecb-a75d-85b6b7264f27/0f4e9512-9bf4-4bde-8f90-172f78a48656"
 					(reference "#PWR03")
