File: modules/SSR/SSR.kicad_sch (KiCad schematic)
At the start: 4 parts, among them J1 Conn_01x08_Pin, J2 Conn_01x16_Socket, J3 Conn_01x01_Pin, J4 Conn_01x09_Pin

Commit message: production output for SSR module
Connections:
- net SSR/AC1 renamed AC7
- net SSR1/AC1 renamed AC6
- net SSR2/AC1 renamed AC5
- net SSR3/AC1 renamed AC4
- net SSR4/AC1 renamed AC3
- net SSR5/AC1 renamed AC2
- net SSR6/AC1 renamed AC1
- net SSR7/AC1 renamed AC0

Commit message: routing
Parts:
- removed J1: Conn_01x08_Pin, Connector_PinHeader_2.54mm:PinHeader_1x08_P2.54mm_Vertical, symbol Connector:Conn_01x08_Pin
- removed J4: Conn_01x09_Pin, Connector_PinHeader_2.54mm:PinHeader_1x09_P2.54mm_Vertical, symbol Connector:Conn_01x09_Pin
- added J1: Conn_01x17_Pin, Connector_PinHeader_2.54mm:PinHeader_1x17_P2.54mm_Vertical, symbol Connector:Conn_01x17_Pin
Connections:
- net AC0: now also J2.1 (Pin_1); no longer J2.8 (Pin_8)
- net AC1: now also J2.2 (Pin_2); no longer J2.7 (Pin_7)
- net AC2: now also J2.3 (Pin_3); no longer J2.6 (Pin_6)
- net AC3: now also J2.4 (Pin_4); no longer J2.5 (Pin_5)
- net AC4: now also J2.5 (Pin_5); no longer J2.4 (Pin_4)
- net AC5: now also J2.6 (Pin_6); no longer J2.3 (Pin_3)
- net AC6: now also J2.7 (Pin_7); no longer J2.2 (Pin_2)
- net AC7: now also J2.8 (Pin_8); no longer J2.1 (Pin_1)
- net GND: now also J1.1 (Pin_1)
- net SSR/Ctrl: now also J1.17 (Pin_17)
- net SSR1/Ctrl: now also J1.16 (Pin_16)
- net SSR10/Ctrl: now also J1.7 (Pin_7)
- net SSR11/Ctrl: now also J1.6 (Pin_6)
- net SSR12/Ctrl: now also J1.5 (Pin_5)
- net SSR13/Ctrl: now also J1.4 (Pin_4)
- net SSR14/Ctrl: now also J1.3 (Pin_3)
- net SSR15/Ctrl: now also J1.2 (Pin_2)
- net SSR2/Ctrl: now also J1.15 (Pin_15)
- net SSR3/Ctrl: now also J1.14 (Pin_14)
- net SSR4/Ctrl: now also J1.13 (Pin_13)
- net SSR5/Ctrl: now also J1.12 (Pin_12)
- net SSR6/Ctrl: now also J1.11 (Pin_11)
- net SSR7/Ctrl: now also J1.10 (Pin_10)
- net SSR8/Ctrl: now also J1.9 (Pin_9)
- net SSR9/Ctrl: now also J1.8 (Pin_8)
Changed lines of the file:
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@@
 	)
 	(label "AC0"
-		(at 166.37 24.13 270)
+		(at 148.59 24.13 270)
 		(effects
 			(font
@@
 	)
 	(label "AC7"
-		(at 148.59 24.13 270)
+		(at 166.37 24.13 270)
 		(effects
 			(font
@@
 	)
 	(label "AC2"
-		(at 161.29 24.13 270)
+		(at 153.67 24.13 270)
 		(effects
 			(font
@@
 	)
 	(label "AC4"
-		(at 156.21 24.13 270)
+		(at 158.75 24.13 270)
 		(effects
 			(font
@@
 	)
 	(label "AC6"
-		(at 151.13 24.13 270)
+		(at 163.83 24.13 270)
 		(effects
 			(font
@@
 	)
 	(label "AC1"
-		(at 163.83 24.13 270)
+		(at 151.13 24.13 270)
 		(effects
 			(font
@@
 	)
 	(label "AC3"
-		(at 158.75 24.13 270)
+		(at 156.21 24.13 270)
 		(effects
 			(font
@@
 	)
 	(label "AC5"
-		(at 153.67 24.13 270)
+		(at 161.29 24.13 270)
 		(effects
 			(font
@@
 	)
 	(symbol
-		(lib_id "Connector:Conn_01x08_Pin")
-		(at 81.28 158.75 90)
+		(lib_id "Connector:Conn_01x17_Pin")
+		(at 93.98 158.75 270)
+		(mirror x)
 		(unit 1)
 		(exclude_from_sim no)
@@
 		(fields_autoplaced yes)
 		(property "Reference" "J1"
-			(at 82.55 160.4193 90)
-			(effects
-				(font
-					(size 1.27 1.27)
-				)
-			)
-		)
-		(property "Value" "Conn_01x08_Pin"
-			(at 82.55 162.8436 90)
-			(effects
-				(font
-					(size 1.27 1.27)
-				)
-			)
-		)
-		(property "Footprint" "Connector_PinHeader_2.54mm:PinHeader_1x08_P2.54mm_Vertical"
-			(at 81.28 158.75 0)
+			(at 93.98 160.4193 90)
+			(effects
+				(font
+					(size 1.27 1.27)
+				)
+			)
+		)
+		(property "Value" "Conn_01x17_Pin"
+			(at 93.98 162.8436 90)
+			(effects
+				(font
+					(size 1.27 1.27)
+				)
+			)
+		)
+		(property "Footprint" "Connector_PinHeader_2.54mm:PinHeader_1x17_P2.54mm_Vertical"
+			(at 93.98 158.75 0)
 			(effects
 				(font
@@
 		)
 		(property "Datasheet" "~"
-			(at 81.28 158.75 0)
-			(effects
-				(font
-					(size 1.27 1.27)
-				)
-				(hide yes)
-			)
-		)
-		(property "Description" "Generic connector, single row, 01x08, script generated"
-			(at 81.28 158.75 0)
-			(effects
-				(font
-					(size 1.27 1.27)
-				)
-				(hide yes)
-			)
-		)
-		(property "LCSC Part #" ""
-			(at 81.28 158.75 90)
-			(effects
-				(font
-					(size 1.27 1.27)
-				)
-				(hide yes)
-			)
+			(at 93.98 158.75 0)
+			(effects
+				(font
+					(size 1.27 1.27)
+				)
+				(hide yes)
+			)
+		)
+		(property "Description" "Generic connector, single row, 01x17, script generated"
+			(at 93.98 158.75 0)
+			(effects
+				(font
+					(size 1.27 1.27)
+				)
+				(hide yes)
+			)
+		)
+		(pin "10"
+		)
+		(pin "16"
+		)
+		(pin "11"
+		)
+		(pin "9"
+		)
+		(pin "15"
+		)
+		(pin "17"
+		)
+		(pin "7"
 		)
 		(pin "8"
 		)
-		(pin "7"
+		(pin "12"
+		)
+		(pin "13"
+		)
+		(pin "14"
+		)
+		(pin "5"
 		)
 		(pin "1"
 		)
+		(pin "4"
+		)
 		(pin "2"
 		)
+		(pin "6"
+		)
 		(pin "3"
 		)
-		(pin "4"
-		)
-		(pin "5"
-		)
-		(pin "6"
-		)
 		(instances
-			(project "SSR"
+			(project ""
 				(path "/e87a2758-91f7-4ecb-a75d-85b6b7264f27"
 					(reference "J1")
 					(unit 1)
 				)
-			)
-		)
-	)
-	(symbol
-		(lib_id "Connector:Conn_01x09_Pin")
-		(at 104.14 158.75 90)
-		(unit 1)
-		(exclude_from_sim no)
-		(in_bom yes)
-		(on_board yes)
-		(dnp no)
-		(fields_autoplaced yes)
-		(property "Reference" "J4"
-			(at 104.14 160.4193 90)
-			(effects
-				(font
-					(size 1.27 1.27)
-				)
-			)
-		)
-		(property "Value" "Conn_01x09_Pin"
-			(at 104.14 162.8436 90)
-			(effects
-				(font
-					(size 1.27 1.27)
-				)
-			)
-		)
-		(property "Footprint" "Connector_PinHeader_2.54mm:PinHeader_1x09_P2.54mm_Vertical"
-			(at 104.14 158.75 0)
-			(effects
-				(font
-					(size 1.27 1.27)
-				)
-				(hide yes)
-			)
-		)
-		(property "Datasheet" "~"
-			(at 104.14 158.75 0)
-			(effects
-				(font
-					(size 1.27 1.27)
-				)
-				(hide yes)
-			)
-		)
-		(property "Description" "Generic connector, single row, 01x09, script generated"
-			(at 104.14 158.75 0)
-			(effects
-				(font
-					(size 1.27 1.27)
-				)
-				(hide yes)
-			)
-		)
-		(property "LCSC Part #" ""
-			(at 104.14 158.75 90)
-			(effects
-				(font
-					(size 1.27 1.27)
-				)
-				(hide yes)
-			)
-		)
-		(pin "3"
-		)
-		(pin "6"
-		)
-		(pin "7"
-		)
-		(pin "9"
-		)
-		(pin "1"
-		)
-		(pin "5"
-		)
-		(pin "4"
-		)
-		(pin "8"
-		)
-		(pin "2"
-		)
-		(instances
-			(project "SSR"
-				(path "/e87a2758-91f7-4ecb-a75d-85b6b7264f27"
-					(reference "J4")
-					(unit 1)
-				)
