File: modules/jkflipflop/nand3.kicad_sch (KiCad schematic)
At the start: 6 parts, among them Q11 AO3401A, Q15 2N7002, Q20 AO3401A, Q3 AO3401A, Q6 2N7002, Q9 2N7002

Commit message: flipflop wip
Parts:
- renumbered Q20 to Q3, Q9 to Q4, Q6 to Q5, Q15 to Q6, Q3 to Q7, Q11 to Q8
