File: modules/jkflipflop/flipflop.kicad_sch (KiCad schematic)
At the start: 1 part

Commit message: flipflop wip
Parts:
- added Q1: AO3401A, Package_TO_SOT_SMD:SOT-23, symbol Transistor_FET:DMP3099L
- added Q2: 2N7002, Package_TO_SOT_SMD:SOT-23, symbol Transistor_FET:2N7002
Connections:
- net +3V3: now also Q1.2 (S)
- net CLK: now also Q1.1 (G), Q2.1 (G)
- net GND: now also Q2.2 (S)
- new net \clk: Q1.3 (D), Q2.3 (D)
Other:
- added sheet NAND2_1 (nand2.kicad_sch)
- added sheet NAND2_2 (nand2.kicad_sch)
- added sheet NAND2_3 (nand2.kicad_sch)
- added sheet NAND2_4 (nand2.kicad_sch)
- moved on the sheet: C1

Commit message: flipflop routing wip
Parts:
- added C5: 100n, Capacitor_SMD:C_0603_1608Metric, symbol Device:C
Connections:
- net +3V3: now also C5.1
- net GND: now also C5.2
Changed lines of the file:
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@@
 	(paper "A4")
 	(junction
+		(at 269.24 99.06)
+		(diameter 0)
+		(color 0 0 0 0)
+	)
+	(junction
 		(at 227.6475 97.7901)
 		(diameter 0)
@@
 	)
 	(junction
+		(at 269.24 91.44)
+		(diameter 0)
+		(color 0 0 0 0)
+	)
+	(junction
+		(at 229.87 97.79)
+		(diameter 0)
+		(color 0 0 0 0)
+	)
+	(junction
+		(at 85.09 83.82)
+		(diameter 0)
+		(color 0 0 0 0)
+	)
+	(junction
+		(at 208.915 77.47)
+		(diameter 0)
+		(color 0 0 0 0)
+	)
+	(junction
+		(at 231.14 85.09)
+		(diameter 0)
+		(color 0 0 0 0)
+	)
+	(junction
+		(at 166.0525 105.41)
+		(diameter 0)
+		(color 0 0 0 0)
+	)
+	(junction
+		(at 143.8275 95.2501)
+		(diameter 0)
+		(color 0 0 0 0)
+	)
+	(junction
+		(at 208.915 73.66)
+		(diameter 0)
+		(color 0 0 0 0)
+	)
+	(junction
 		(at 166.0525 97.79)
 		(diameter 0)
@@
 	)
 	(junction
-		(at 229.87 97.79)
-		(diameter 0)
-		(color 0 0 0 0)
-	)
-	(junction
-		(at 85.09 83.82)
-		(diameter 0)
-		(color 0 0 0 0)
-	)
-	(junction
-		(at 208.915 77.47)
-		(diameter 0)
-		(color 0 0 0 0)
-	)
-	(junction
-		(at 231.14 85.09)
-		(diameter 0)
-		(color 0 0 0 0)
-	)
-	(junction
-		(at 166.0525 105.41)
-		(diameter 0)
-		(color 0 0 0 0)
-	)
-	(junction
-		(at 143.8275 95.2501)
-		(diameter 0)
-		(color 0 0 0 0)
-	)
-	(junction
-		(at 208.915 73.66)
-		(diameter 0)
-		(color 0 0 0 0)
-	)
-	(junction
 		(at 125.095 71.12)
 		(diameter 0)
@@
 	(wire
 		(pts
-			(xy 166.0525 97.79) (xy 160.02 97.79)
-		)
-		(stroke
-			(width 0)
-			(type default)
-		)
-	)
-	(wire
-		(pts
-			(xy 166.37 97.79) (xy 166.0525 97.79)
+			(xy 160.02 105.41) (xy 166.0525 105.41)
 		)
 		(stroke
@@
 	(wire
 		(pts
+			(xy 165.1 97.79) (xy 166.0525 97.79)
+		)
+		(stroke
+			(width 0)
+			(type default)
+		)
+	)
+	(wire
+		(pts
 			(xy 208.915 73.66) (xy 209.55 73.66)
 		)
@@
 	(wire
 		(pts
+			(xy 269.24 99.06) (xy 279.4 99.06)
+		)
+		(stroke
+			(width 0)
+			(type default)
+		)
+	)
+	(wire
+		(pts
 			(xy 226.06 74.93) (xy 226.3775 74.93)
 		)
@@
 	(wire
 		(pts
-			(xy 85.09 92.71) (xy 88.9 92.71)
-		)
-		(stroke
-			(width 0)
-			(type default)
-		)
-	)
-	(wire
-		(pts
 			(xy 142.5575 72.39) (xy 147.32 72.39)
 		)
@@
 	(wire
 		(pts
+			(xy 85.09 100.33) (xy 88.9 100.33)
+		)
+		(stroke
+			(width 0)
+			(type default)
+		)
+	)
+	(wire
+		(pts
 			(xy 208.915 77.47) (xy 209.55 77.47)
 		)
@@
 	(wire
 		(pts
-			(xy 85.09 92.71) (xy 85.09 83.82)
+			(xy 85.09 83.82) (xy 85.09 100.33)
 		)
 		(stroke
@@
 	(wire
 		(pts
+			(xy 166.0525 97.79) (xy 166.37 97.79)
+		)
+		(stroke
+			(width 0)
+			(type default)
+		)
+	)
+	(wire
+		(pts
 			(xy 166.0525 101.6) (xy 146.05 101.6)
 		)
@@
 	(wire
 		(pts
-			(xy 81.28 100.33) (xy 88.9 100.33)
-		)
-		(stroke
-			(width 0)
-			(type default)
-		)
-	)
-	(wire
-		(pts
-			(xy 165.1 105.41) (xy 166.0525 105.41)
+			(xy 269.24 91.44) (xy 279.4 91.44)
+		)
+		(stroke
+			(width 0)
+			(type default)
+		)
+	)
+	(wire
+		(pts
+			(xy 81.28 92.71) (xy 88.9 92.71)
 		)
 		(stroke
@@
 	)
 	(label "\\clk"
-		(at 160.02 97.79 180)
+		(at 160.02 105.41 180)
 		(effects
 			(font
@@
 	(hierarchical_label "Preset"
 		(shape input)
-		(at 165.1 105.41 180)
+		(at 165.1 97.79 180)
 		(effects
 			(font
@@
 	(hierarchical_label "K"
 		(shape input)
-		(at 81.28 100.33 180)
+		(at 81.28 92.71 180)
 		(effects
 			(font
@@
 					(unit 1)
 				)
+			)
+		)
+	)
+	(symbol
+		(lib_id "Device:C")
+		(at 279.4 95.25 0)
+		(unit 1)
+		(exclude_from_sim no)
+		(in_bom yes)
+		(on_board yes)
+		(dnp no)
+		(fields_autoplaced yes)
+		(property "Reference" "C5"
+			(at 282.321 94.0378 0)
+			(effects
+				(font
+					(size 1.27 1.27)
+				)
+				(justify left)
+			)
+		)
+		(property "Value" "100n"
+			(at 282.321 96.4621 0)
+			(effects
+				(font
+					(size 1.27 1.27)
+				)
+				(justify left)
+			)
+		)
+		(property "Footprint" "Capacitor_SMD:C_0603_1608Metric"
+			(at 280.3652 99.06 0)
+			(effects
+				(font
+					(size 1.27 1.27)
+				)
+				(hide yes)
+			)
+		)
+		(property "Datasheet" "~"
+			(at 279.4 95.25 0)
+			(effects
+				(font
+					(size 1.27 1.27)
+				)
+				(hide yes)
+			)
+		)
+		(property "Description" "Unpolarized capacitor"
+			(at 279.4 95.25 0)
+			(effects
+				(font
+					(size 1.27 1.27)
+				)
+				(hide yes)
+			)
+		)
+		(property "LCSC Part #" "C14663"
+			(at 279.4 95.25 0)
+			(effects
+				(font
+					(size 1.27 1.27)
+				)
+				(hide yes)
+			)
+		)
+		(pin "2"
+		)
+		(pin "1"
+		)
+		(instances
+			(project "jkflipflop"
+				(path "/8013391e-c8e7-41ee-accd-360f92f3a5d7/259d22b3-bbdc-4d1c-a30b-6746a4fa5b6c"
+					(reference "C7")
+					(unit 1)
+				)
+				(path "/8013391e-c8e7-41ee-accd-360f92f3a5d7/6979d884-3104-4d4d-a14e-0e449b6f5d88"
+					(reference "C5")
+					(unit 1)
+				)
+				(path "/8013391e-c8e7-41ee-accd-360f92f3a5d7/9318a685-33db-476b-a8fe-85a58a155206"
+					(reference "C6")
+					(unit 1)
+				)
+				(path "/8013391e-c8e7-41ee-accd-360f92f3a5d7/caa3c691-168b-4b9f-bbf3-d1a553e02d69"
+					(reference "C8")
+					(unit 1)
+				)
