File: modules/jkflipflop/jkflipflop.kicad_sch (KiCad schematic)
At the start: 1 part, among them J1 Conn_02x26_Odd_Even

Commit message: routed flipflops
Connections:
- net jk-flipflop/CLK: now also J1.23 (Pin_23); no longer J1.14 (Pin_14)
- net jk-flipflop/Clr: now also J1.29 (Pin_29); no longer J1.2 (Pin_2)
- net jk-flipflop/J: now also J1.21 (Pin_21); no longer J1.12 (Pin_12)
- net jk-flipflop/K: now also J1.25 (Pin_25); no longer J1.16 (Pin_16)
- net jk-flipflop/Preset: now also J1.35 (Pin_35); no longer J1.8 (Pin_8)
- net jk-flipflop/Q: now also J1.31 (Pin_31); no longer J1.4 (Pin_4)
- net jk-flipflop/\Q: now also J1.33 (Pin_33); no longer J1.6 (Pin_6)
- net jk-flipflop1/CLK: now also J1.14 (Pin_14); no longer J1.32 (Pin_32)
- net jk-flipflop1/Clr: now also J1.2 (Pin_2); no longer J1.20 (Pin_20)
- net jk-flipflop1/J: now also J1.12 (Pin_12); no longer J1.30 (Pin_30)
- net jk-flipflop1/K: now also J1.16 (Pin_16); no longer J1.34 (Pin_34)
- net jk-flipflop1/Preset: now also J1.8 (Pin_8); no longer J1.26 (Pin_26)
- net jk-flipflop1/Q: now also J1.4 (Pin_4); no longer J1.22 (Pin_22)
- net jk-flipflop1/\Q: now also J1.6 (Pin_6); no longer J1.24 (Pin_24)
- net jk-flipflop3/CLK: now also J1.32 (Pin_32); no longer J1.23 (Pin_23)
- net jk-flipflop3/Clr: now also J1.20 (Pin_20); no longer J1.29 (Pin_29)
- net jk-flipflop3/J: now also J1.30 (Pin_30); no longer J1.21 (Pin_21)
- net jk-flipflop3/K: now also J1.34 (Pin_34); no longer J1.25 (Pin_25)
- net jk-flipflop3/Preset: now also J1.26 (Pin_26); no longer J1.35 (Pin_35)
- net jk-flipflop3/Q: now also J1.24 (Pin_24); no longer J1.33 (Pin_33)
- net jk-flipflop3/\Q: now also J1.22 (Pin_22); no longer J1.31 (Pin_31)
Changed lines of the file:
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@@
+	)
+	(sheet
+		(at 50.8 152.4)
+		(size 20.32 16.51)
+		(exclude_from_sim no)
+		(in_bom yes)
+		(on_board yes)
+		(dnp no)
+		(fields_autoplaced yes)
+		(stroke
+			(width 0.1524)
+			(type solid)
+		)
+		(fill
+			(color 0 0 0 0.0000)
+		)
+		(property "Sheetname" "jk-flipflop1"
+			(at 50.8 151.6884 0)
+			(effects
+				(font
+					(size 1.27 1.27)
+				)
+				(justify left bottom)
+			)
+		)
+		(property "Sheetfile" "flipflop.kicad_sch"
+			(at 50.8 169.4946 0)
+			(effects
+				(font
+					(size 1.27 1.27)
+				)
+				(justify left top)
+			)
+		)
+		(pin "CLK" input
+			(at 71.12 160.02 0)
+			(effects
+				(font
+					(size 1.27 1.27)
+				)
+				(justify right)
+			)
+		)
+		(pin "Clr" input
+			(at 50.8 166.37 180)
+			(effects
+				(font
+					(size 1.27 1.27)
+				)
+				(justify left)
+			)
+		)
+		(pin "J" input
+			(at 71.12 156.21 0)
+			(effects
+				(font
+					(size 1.27 1.27)
+				)
+				(justify right)
+			)
+		)
+		(pin "K" input
+			(at 71.12 163.83 0)
+			(effects
+				(font
+					(size 1.27 1.27)
+				)
+				(justify right)
+			)
+		)
+		(pin "Preset" input
+			(at 50.8 154.94 180)
+			(effects
+				(font
+					(size 1.27 1.27)
+				)
+				(justify left)
+			)
+		)
+		(pin "Q" output
+			(at 50.8 162.56 180)
+			(effects
+				(font
+					(size 1.27 1.27)
+				)
+				(justify left)
+			)
+		)
+		(pin "\\Q" output
+			(at 50.8 158.75 180)
+			(effects
+				(font
+					(size 1.27 1.27)
+				)
+				(justify left)
+			)
+		)
+		(instances
+			(project "jkflipflop"
+				(path "/8013391e-c8e7-41ee-accd-360f92f3a5d7"
+					(page "2")
+				)
+			)
+		)
+	)
+	(sheet
+		(at 114.3 55.88)
+		(size 20.32 16.51)
+		(exclude_from_sim no)
+		(in_bom yes)
+		(on_board yes)
+		(dnp no)
+		(fields_autoplaced yes)
+		(stroke
+			(width 0.1524)
+			(type solid)
+		)
+		(fill
+			(color 0 0 0 0.0000)
+		)
+		(property "Sheetname" "jk-flipflop"
+			(at 114.3 55.1684 0)
+			(effects
+				(font
+					(size 1.27 1.27)
+				)
+				(justify left bottom)
+			)
+		)
+		(property "Sheetfile" "flipflop.kicad_sch"
+			(at 114.3 72.9746 0)
+			(effects
+				(font
+					(size 1.27 1.27)
+				)
+				(justify left top)
+			)
+		)
+		(pin "CLK" input
+			(at 114.3 63.5 180)
+			(effects
+				(font
+					(size 1.27 1.27)
+				)
+				(justify left)
+			)
+		)
+		(pin "Clr" input
+			(at 134.62 69.85 0)
+			(effects
+				(font
+					(size 1.27 1.27)
+				)
+				(justify right)
+			)
+		)
+		(pin "J" input
+			(at 114.3 59.69 180)
+			(effects
+				(font
+					(size 1.27 1.27)
+				)
+				(justify left)
+			)
+		)
+		(pin "K" input
+			(at 114.3 67.31 180)
+			(effects
+				(font
+					(size 1.27 1.27)
+				)
+				(justify left)
+			)
+		)
+		(pin "Preset" input
+			(at 134.62 58.42 0)
+			(effects
+				(font
+					(size 1.27 1.27)
+				)
+				(justify right)
+			)
+		)
+		(pin "Q" output
+			(at 134.62 66.04 0)
+			(effects
+				(font
+					(size 1.27 1.27)
+				)
+				(justify right)
+			)
+		)
+		(pin "\\Q" output
+			(at 134.62 62.23 0)
+			(effects
+				(font
+					(size 1.27 1.27)
+				)
+				(justify right)
+			)
+		)
+		(instances
+			(project "jkflipflop"
+				(path "/8013391e-c8e7-41ee-accd-360f92f3a5d7"
+					(page "6")
+				)
+			)
+		)
 	)
 	(sheet
@@
 			(color 0 0 0 0.0000)
 		)
-		(property "Sheetname" "jk-flipflop1"
+		(property "Sheetname" "jk-flipflop3"
 			(at 110.49 152.9584 0)
 			(effects
@@
 		)
 		(pin "Q" output
+			(at 110.49 160.02 180)
+			(effects
+				(font
+					(size 1.27 1.27)
+				)
+				(justify left)
+			)
+		)
+		(pin "\\Q" output
 			(at 110.49 163.83 180)
 			(effects
@@
 			)
 		)
-		(pin "\\Q" output
-			(at 110.49 160.02 180)
-			(effects
-				(font
-					(size 1.27 1.27)
-				)
-				(justify left)
-			)
-		)
-		(instances
-			(project "jkflipflop"
-				(path "/8013391e-c8e7-41ee-accd-360f92f3a5d7"
-					(page "2")
-				)
-			)
-		)
-	)
-	(sheet
-		(at 50.8 152.4)
-		(size 20.32 16.51)
-		(exclude_from_sim no)
-		(in_bom yes)
-		(on_board yes)
-		(dnp no)
-		(fields_autoplaced yes)
-		(stroke
-			(width 0.1524)
-			(type solid)
-		)
-		(fill
-			(color 0 0 0 0.0000)
-		)
-		(property "Sheetname" "jk-flipflop"
-			(at 50.8 151.6884 0)
-			(effects
-				(font
-					(size 1.27 1.27)
-				)
-				(justify left bottom)
-			)
-		)
-		(property "Sheetfile" "flipflop.kicad_sch"
-			(at 50.8 169.4946 0)
-			(effects
-				(font
-					(size 1.27 1.27)
-				)
-				(justify left top)
-			)
-		)
-		(pin "CLK" input
-			(at 71.12 160.02 0)
-			(effects
-				(font
-					(size 1.27 1.27)
-				)
-				(justify right)
-			)
-		)
-		(pin "Clr" input
-			(at 50.8 166.37 180)
-			(effects
-				(font
-					(size 1.27 1.27)
-				)
-				(justify left)
-			)
-		)
-		(pin "J" input
-			(at 71.12 156.21 0)
-			(effects
-				(font
-					(size 1.27 1.27)
-				)
-				(justify right)
-			)
-		)
-		(pin "K" input
-			(at 71.12 163.83 0)
-			(effects
-				(font
-					(size 1.27 1.27)
-				)
-				(justify right)
-			)
-		)
-		(pin "Preset" input
-			(at 50.8 154.94 180)
-			(effects
-				(font
-					(size 1.27 1.27)
-				)
-				(justify left)
-			)
-		)
-		(pin "Q" output
-			(at 50.8 162.56 180)
-			(effects
-				(font
-					(size 1.27 1.27)
-				)
-				(justify left)
-			)
-		)
-		(pin "\\Q" output
-			(at 50.8 158.75 180)
-			(effects
-				(font
-					(size 1.27 1.27)
-				)
-				(justify left)
-			)
-		)
-		(instances
-			(project "jkflipflop"
-				(path "/8013391e-c8e7-41ee-accd-360f92f3a5d7"
-					(page "6")
-				)
-			)
-		)
-	)
-	(sheet
-		(at 114.3 55.88)
-		(size 20.32 16.51)
-		(exclude_from_sim no)
-		(in_bom yes)
-		(on_board yes)
-		(dnp no)
-		(fields_autoplaced yes)
-		(stroke
-			(width 0.1524)
-			(type solid)
-		)
-		(fill
-			(color 0 0 0 0.0000)
-		)
-		(property "Sheetname" "jk-flipflop3"
-			(at 114.3 55.1684 0)
-			(effects
-				(font
-					(size 1.27 1.27)
-				)
-				(justify left bottom)
-			)
-		)
-		(property "Sheetfile" "flipflop.kicad_sch"
-			(at 114.3 72.9746 0)
-			(effects
-				(font
-					(size 1.27 1.27)
-				)
-				(justify left top)
-			)
-		)
-		(pin "CLK" input
-			(at 114.3 63.5 180)
-			(effects
-				(font
-					(size 1.27 1.27)
-				)
-				(justify left)
-			)
-		)
-		(pin "Clr" input
-			(at 134.62 69.85 0)
-			(effects
-				(font
-					(size 1.27 1.27)
-				)
-				(justify right)
-			)
-		)
-		(pin "J" input
-			(at 114.3 59.69 180)
-			(effects
-				(font
-					(size 1.27 1.27)
-				)
-				(justify left)
-			)
-		)
-		(pin "K" input
-			(at 114.3 67.31 180)
-			(effects
-				(font
-					(size 1.27 1.27)
-				)
-				(justify left)
-			)
-		)
-		(pin "Preset" input
-			(at 134.62 58.42 0)
-			(effects
-				(font
-					(size 1.27 1.27)
-				)
-				(justify right)
-			)
-		)
-		(pin "Q" output
-			(at 134.62 62.23 0)
-			(effects
-				(font
-					(size 1.27 1.27)
-				)
-				(justify right)
-			)
-		)
-		(pin "\\Q" output
-			(at 134.62 66.04 0)
-			(effects
-				(font
-					(size 1.27 1.27)
-				)
-				(justify right)
-			)
-		)
