File: modules/jkflipflop/jkflipflop.kicad_pcb (KiCad board)
At the start: 2 copper layers, 57.2 x 61.2 mm, 101 parts, among them J1 Conn_02x26_Odd_Even, Q1 2N7002, Q10 2N7002, Q11 AO3401A, Q12 2N7002, Q13 2N7002, Q14 AO3401A, Q15 2N7002, Q16 AO3401A, Q17 2N7002, Q18 AO3401A, Q19 AO3401A, Q2 2N7002, Q20 AO3401A, Q21 AO3401A, Q22 2N7002, Q23 2N7002, Q24 AO3401A, Q25 2N7002, Q26 2N7002, Q27 AO3401A, Q28 AO3401A, Q29 2N7002, Q3 AO3401A, Q30 AO3401A, Q31 AO3401A, Q32 AO3401A, Q33 2N7002, Q34 AO3401A, Q35 2N7002, Q36 2N7002, Q37 2N7002, Q38 AO3401A, Q39 AO3401A, Q4 AO3401A, Q40 2N7002, Q41 2N7002, Q42 AO3401A, Q43 AO3401A, Q44 AO3401A, Q45 2N7002, Q46 2N7002, Q47 2N7002, Q48 2N7002, Q49 AO3401A, Q5 AO3401A, Q50 2N7002, Q51 AO3401A, Q52 2N7002, Q53 AO3401A, Q54 AO3401A, Q55 AO3401A, Q56 AO3401A, Q57 AO3401A, Q58 2N7002, Q59 2N7002, Q6 2N7002, Q60 2N7002, Q61 2N7002, Q62 AO3401A, Q63 2N7002, Q64 2N7002, Q65 AO3401A, Q66 AO3401A, Q67 2N7002, Q68 AO3401A, Q69 2N7002, Q7 2N7002, Q70 AO3401A, Q71 AO3401A, Q72 2N7002, Q73 AO3401A, Q74 AO3401A, Q75 AO3401A, Q76 2N7002, Q77 2N7002, Q78 2N7002, Q79 AO3401A, Q8 AO3401A, Q80 2N7002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

Commit message: flipflop wip
Parts:
- added Q100: 2N7002, Package_TO_SOT_SMD:SOT-23, F.Cu at (354.0, 40.3)
- added Q101: AO3401A, Package_TO_SOT_SMD:SOT-23, F.Cu at (358.1, 43.8)
- added Q102: AO3401A, Package_TO_SOT_SMD:SOT-23, F.Cu at (354.0, 36.8)
- added Q103: AO3401A, Package_TO_SOT_SMD:SOT-23, F.Cu at (242.1, 40.5)
- added Q104: AO3401A, Package_TO_SOT_SMD:SOT-23, F.Cu at (110.2, 152.7)
- added Q105: 2N7002, Package_TO_SOT_SMD:SOT-23, F.Cu at (242.1, 44.0)
- added Q106: 2N7002, Package_TO_SOT_SMD:SOT-23, F.Cu at (238.0, 47.5)
- added Q107: 2N7002, Package_TO_SOT_SMD:SOT-23, F.Cu at (238.0, 44.0)
- added Q108: 2N7002, Package_TO_SOT_SMD:SOT-23, F.Cu at (110.2, 156.2)
- added Q109: 2N7002, Package_TO_SOT_SMD:SOT-23, F.Cu at (114.3, 156.2)
- added Q110: AO3401A, Package_TO_SOT_SMD:SOT-23, F.Cu at (242.1, 47.5)
- added Q111: AO3401A, Package_TO_SOT_SMD:SOT-23, F.Cu at (114.3, 152.7)
- added Q112: AO3401A, Package_TO_SOT_SMD:SOT-23, F.Cu at (237.9, 40.5)
- added Q113: AO3401A, Package_TO_SOT_SMD:SOT-23, F.Cu at (96.4, 172.5)
- added Q114: 2N7002, Package_TO_SOT_SMD:SOT-23, F.Cu at (96.4, 176.0)
- added Q115: 2N7002, Package_TO_SOT_SMD:SOT-23, F.Cu at (100.5, 176.0)
- added Q116: AO3401A, Package_TO_SOT_SMD:SOT-23, F.Cu at (100.5, 172.5)
- added Q117: AO3401A, Package_TO_SOT_SMD:SOT-23, F.Cu at (272.7, 66.5)
- added Q118: 2N7002, Package_TO_SOT_SMD:SOT-23, F.Cu at (272.7, 70.0)
- added Q119: 2N7002, Package_TO_SOT_SMD:SOT-23, F.Cu at (276.8, 70.0)
- added Q120: AO3401A, Package_TO_SOT_SMD:SOT-23, F.Cu at (276.8, 66.5)
- added Q121: AO3401A, Package_TO_SOT_SMD:SOT-23, F.Cu at (355.6, 76.5)
- added Q122: 2N7002, Package_TO_SOT_SMD:SOT-23, F.Cu at (355.6, 80.0)
- added Q123: 2N7002, Package_TO_SOT_SMD:SOT-23, F.Cu at (359.7, 80.0)
- added Q124: AO3401A, Package_TO_SOT_SMD:SOT-23, F.Cu at (359.7, 76.5)
- added Q125: AO3401A, Package_TO_SOT_SMD:SOT-23, F.Cu at (430.2, 168.4)
- added Q126: 2N7002, Package_TO_SOT_SMD:SOT-23, F.Cu at (430.2, 171.9)
- added Q127: 2N7002, Package_TO_SOT_SMD:SOT-23, F.Cu at (434.3, 171.9)
- added Q128: AO3401A, Package_TO_SOT_SMD:SOT-23, F.Cu at (434.3, 168.4)
- added Q129: AO3401A, Package_TO_SOT_SMD:SOT-23, F.Cu at (407.3, 167.8)
- added Q130: 2N7002, Package_TO_SOT_SMD:SOT-23, F.Cu at (407.4, 171.3)
- added Q131: 2N7002, Package_TO_SOT_SMD:SOT-23, F.Cu at (411.5, 171.3)
- added Q132: AO3401A, Package_TO_SOT_SMD:SOT-23, F.Cu at (411.5, 167.8)
- added Q133: AO3401A, Package_TO_SOT_SMD:SOT-23, F.Cu at (149.2, 149.1)
- added Q134: 2N7002, Package_TO_SOT_SMD:SOT-23, F.Cu at (149.2, 152.6)
- added Q135: 2N7002, Package_TO_SOT_SMD:SOT-23, F.Cu at (153.3, 152.6)
- added Q136: AO3401A, Package_TO_SOT_SMD:SOT-23, F.Cu at (153.3, 149.1)
- added Q137: AO3401A, Package_TO_SOT_SMD:SOT-23, F.Cu at (162.2, 190.0)
- added Q138: 2N7002, Package_TO_SOT_SMD:SOT-23, F.Cu at (162.3, 193.5)
- added Q139: 2N7002, Package_TO_SOT_SMD:SOT-23, F.Cu at (166.4, 193.5)
- added Q140: AO3401A, Package_TO_SOT_SMD:SOT-23, F.Cu at (166.4, 190.0)
- added Q141: AO3401A, Package_TO_SOT_SMD:SOT-23, F.Cu at (224.3, 86.3)
- added Q142: 2N7002, Package_TO_SOT_SMD:SOT-23, F.Cu at (224.3, 89.8)
- added Q143: 2N7002, Package_TO_SOT_SMD:SOT-23, F.Cu at (228.4, 89.8)
- added Q144: AO3401A, Package_TO_SOT_SMD:SOT-23, F.Cu at (228.4, 86.3)
- added Q145: AO3401A, Package_TO_SOT_SMD:SOT-23, F.Cu at (279.7, 101.1)
- added Q146: 2N7002, Package_TO_SOT_SMD:SOT-23, F.Cu at (279.7, 104.6)
- added Q147: 2N7002, Package_TO_SOT_SMD:SOT-23, F.Cu at (283.8, 104.6)
- added Q148: AO3401A, Package_TO_SOT_SMD:SOT-23, F.Cu at (283.8, 101.1)
- added Q149: AO3401A, Package_TO_SOT_SMD:SOT-23, F.Cu at (329.6, 81.4)
- added Q150: 2N7002, Package_TO_SOT_SMD:SOT-23, F.Cu at (329.6, 84.9)
- added Q151: 2N7002, Package_TO_SOT_SMD:SOT-23, F.Cu at (333.7, 84.9)
- added Q152: AO3401A, Package_TO_SOT_SMD:SOT-23, F.Cu at (333.7, 81.4)
- added Q153: AO3401A, Package_TO_SOT_SMD:SOT-23, F.Cu at (402.9, 60.2)
- added Q154: 2N7002, Package_TO_SOT_SMD:SOT-23, F.Cu at (402.9, 63.7)
- added Q155: 2N7002, Package_TO_SOT_SMD:SOT-23, F.Cu at (407.0, 63.7)
- added Q156: AO3401A, Package_TO_SOT_SMD:SOT-23, F.Cu at (407.0, 60.2)
- added Q157: AO3401A, Package_TO_SOT_SMD:SOT-23, F.Cu at (390.5, 167.8)
- added Q158: 2N7002, Package_TO_SOT_SMD:SOT-23, F.Cu at (390.5, 171.3)
- added Q159: 2N7002, Package_TO_SOT_SMD:SOT-23, F.Cu at (394.6, 171.3)
- added Q160: AO3401A, Package_TO_SOT_SMD:SOT-23, F.Cu at (394.6, 167.8)
- added Q161: AO3401A, Package_TO_SOT_SMD:SOT-23, F.Cu at (401.9, 34.5)
- added Q162: 2N7002, Package_TO_SOT_SMD:SOT-23, F.Cu at (402.0, 37.9)
- added Q163: 2N7002, Package_TO_SOT_SMD:SOT-23, F.Cu at (406.1, 37.9)
- added Q164: AO3401A, Package_TO_SOT_SMD:SOT-23, F.Cu at (406.1, 34.5)
- added Q165: AO3401A, Package_TO_SOT_SMD:SOT-23, F.Cu at (238.1, 86.3)
- added Q166: 2N7002, Package_TO_SOT_SMD:SOT-23, F.Cu at (238.2, 89.8)
- added Q167: 2N7002, Package_TO_SOT_SMD:SOT-23, F.Cu at (242.2, 89.8)
- added Q168: AO3401A, Package_TO_SOT_SMD:SOT-23, F.Cu at (242.2, 86.3)
- added Q97: AO3401A, Package_TO_SOT_SMD:SOT-23, F.Cu at (358.1, 36.8)
- added Q98: 2N7002, Package_TO_SOT_SMD:SOT-23, F.Cu at (358.2, 40.3)
- added Q99: 2N7002, Package_TO_SOT_SMD:SOT-23, F.Cu at (354.0, 43.8)
- Q1, Q13, Q15, Q23, Q29, Q33, Q35, Q40, Q41, Q45, Q46, Q47, Q52, Q59, Q63, Q64, Q69, Q7, Q76, Q77, Q83, Q9, Q90, Q91, Q95: value 2N7002 -> AO3401A
- Q11, Q16, Q18, Q24, Q30, Q31, Q32, Q38, Q4, Q42, Q43, Q44, Q49, Q5, Q54, Q55, Q62, Q66, Q68, Q73, Q74, Q82, Q87, Q93, Q94: value AO3401A -> 2N7002
- moved Q7 365.2 mm to (412.9, 205.8)
- moved Q51 364.8 mm to (432.0, 205.8), turned to 0 degrees
- moved Q4 360.1 mm to (412.9, 202.3)
- moved Q47 357.5 mm to (432.0, 198.8), turned to 0 degrees
- moved Q6 356.6 mm to (408.8, 202.3)
- moved Q8 356.3 mm to (408.7, 198.8)
- moved Q5 356.3 mm to (408.8, 205.8)
- moved Q3 355.3 mm to (412.9, 198.8)
- moved Q48 352.8 mm to (432.0, 202.3)
- moved Q50 347.6 mm to (427.8, 202.3)
- moved Q49 345.3 mm to (427.8, 205.8)
- moved Q52 337.4 mm to (427.8, 198.8), turned to 0 degrees
- moved Q2 335.1 mm to (381.7, 197.7)
- moved Q1 330.2 mm to (381.7, 193.3)
- moved C1 326.4 mm to (386.2, 192.3), turned to 0 degrees
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Connections:
- Q1 pad 2: GND -> +3V3
- Q1 pad 3: Net-(Q1-D) -> /jk-flipflop1/\clk
- Q10 pad 1: /jk-flipflop4/Clr -> /jk-flipflop1/J
- Q10 pad 2: GND -> Net-(Q10-S)
- Q10 pad 3: Net-(Q10-D) -> /jk-flipflop1/NAND2_1/A
- Q11 pad 1: /jk-flipflop1/K -> /jk-flipflop1/\Q
- Q11 pad 2: +3V3 -> Net-(Q11-S)
- Q11 pad 3: /jk-flipflop1/NAND3_2/Out -> Net-(Q10-S)
- Q12 pad 1: /jk-flipflop4/NAND3_2/Out -> /jk-flipflop1/CLK
- Q12 pad 2: Net-(Q10-D) -> GND
- Q12 pad 3: Net-(Q12-D) -> Net-(Q11-S)
- Q13 pad 1: /jk-flipflop4/\Q -> /jk-flipflop1/\Q
- Q13 pad 2: GND -> +3V3
- Q13 pad 3: Net-(Q13-D) -> /jk-flipflop1/NAND2_1/A
- Q14 pad 1: /jk-flipflop4/NAND3_2/Out -> /jk-flipflop1/CLK
- Q14 pad 3: /jk-flipflop4/\Q -> /jk-flipflop1/NAND2_1/A
- Q15 pad 1: /jk-flipflop1/K -> /jk-flipflop1/Clr
- Q15 pad 2: GND -> +3V3
- Q15 pad 3: Net-(Q15-D) -> /jk-flipflop1/NAND2_3/A
- Q16 pad 1: /jk-flipflop4/Clr -> /jk-flipflop1/Clr
- Q16 pad 2: +3V3 -> Net-(Q16-S)
- Q16 pad 3: /jk-flipflop4/\Q -> /jk-flipflop1/NAND2_3/A
- Q17 pad 1: /jk-flipflop4/Q -> /jk-flipflop1/NAND2_1/Out
- Q17 pad 2: Net-(Q12-D) -> Net-(Q17-S)
- Q17 pad 3: /jk-flipflop4/\Q -> Net-(Q16-S)
- Q18 pad 1: /jk-flipflop4/Q -> /jk-flipflop1/\clk
- Q18 pad 2: +3V3 -> GND
- Q18 pad 3: /jk-flipflop4/\Q -> Net-(Q17-S)
- Q19 pad 1: /jk-flipflop4/\Q -> /jk-flipflop1/NAND2_1/Out
- Q19 pad 3: /jk-flipflop4/Q -> /jk-flipflop1/NAND2_3/A
- Q2 pad 1: /jk-flipflop1/\Q -> /jk-flipflop1/CLK
- Q2 pad 2: Net-(Q1-D) -> GND
- Q2 pad 3: Net-(Q2-D) -> /jk-flipflop1/\clk
- Q20 pad 1: /jk-flipflop1/CLK -> /jk-flipflop1/\clk
- Q20 pad 3: /jk-flipflop1/NAND3_2/Out -> /jk-flipflop1/NAND2_3/A
- Q21 pad 1: /jk-flipflop4/Preset -> /jk-flipflop/CLK
- Q21 pad 3: /jk-flipflop4/Q -> /jk-flipflop/\clk
- Q22 pad 1: /jk-flipflop4/Preset -> /jk-flipflop/CLK
- Q22 pad 2: Net-(Q22-S) -> GND
- Q22 pad 3: /jk-flipflop4/Q -> /jk-flipflop/\clk
- Q23 pad 1: /jk-flipflop4/NAND3_1/Out -> /jk-flipflop/J
- Q23 pad 2: Net-(Q13-D) -> +3V3
- Q23 pad 3: Net-(Q22-S) -> /jk-flipflop/NAND2_1/A
- Q24 pad 1: /jk-flipflop4/NAND3_1/Out -> /jk-flipflop/J
- Q24 pad 2: +3V3 -> Net-(Q24-S)
- Q24 pad 3: /jk-flipflop4/Q -> /jk-flipflop/NAND2_1/A
- Q25 pad 3: Net-(Q25-D) -> Net-(Q24-S)
- Q27 pad 1: /jk-flipflop1/NAND3_2/Out -> /jk-flipflop/\Q
- Q27 pad 3: /jk-flipflop1/\Q -> /jk-flipflop/NAND2_1/A
- Q28 pad 3: /jk-flipflop/NAND3_1/Out -> /jk-flipflop/NAND2_1/A
- Q29 pad 1: /jk-flipflop1/\Q -> /jk-flipflop/CLK
- Q29 pad 2: GND -> +3V3
- Q29 pad 3: Net-(Q29-D) -> /jk-flipflop/NAND2_2/B
- Q3 pad 1: /jk-flipflop1/Q -> /jk-flipflop1/CLK
- Q3 pad 3: /jk-flipflop1/NAND3_2/Out -> /jk-flipflop1/NAND2_2/B
- Q30 pad 1: /jk-flipflop/\Q -> /jk-flipflop/CLK
- Q30 pad 2: +3V3 -> Net-(Q30-S)
- Q30 pad 3: /jk-flipflop/NAND3_1/Out -> /jk-flipflop/NAND2_2/B
- Q31 pad 1: /jk-flipflop1/\Q -> /jk-flipflop/Q
- Q31 pad 2: +3V3 -> Net-(Q31-S)
- Q31 pad 3: /jk-flipflop1/Q -> Net-(Q30-S)
- Q32 pad 1: /jk-flipflop/Q -> /jk-flipflop/K
- Q32 pad 2: +3V3 -> GND
- Q32 pad 3: /jk-flipflop/NAND3_2/Out -> Net-(Q31-S)
- Q33 pad 1: /jk-flipflop1/Preset -> /jk-flipflop/Q
- Q33 pad 2: Net-(Q33-S) -> +3V3
- Q33 pad 3: /jk-flipflop1/Q -> /jk-flipflop/NAND2_2/B
- Q34 pad 1: /jk-flipflop1/Preset -> /jk-flipflop/K
- Q34 pad 3: /jk-flipflop1/Q -> /jk-flipflop/NAND2_2/B
- Q35 pad 1: /jk-flipflop1/NAND3_2/Out -> /jk-flipflop/Clr
- Q35 pad 2: Net-(Q35-S) -> +3V3
- Q35 pad 3: Net-(Q35-D) -> /jk-flipflop/NAND2_3/A
- Q36 pad 1: /jk-flipflop1/NAND3_1/Out -> /jk-flipflop/Clr
- Q36 pad 2: Net-(Q29-D) -> Net-(Q36-S)
- Q36 pad 3: Net-(Q33-S) -> /jk-flipflop/NAND2_3/A
- Q37 pad 1: /jk-flipflop/Q -> /jk-flipflop/NAND2_1/Out
- Q37 pad 3: Net-(Q37-D) -> Net-(Q36-S)
- Q38 pad 1: /jk-flipflop/J -> /jk-flipflop/\clk
- Q38 pad 2: +3V3 -> GND
- Q38 pad 3: /jk-flipflop/NAND3_1/Out -> Net-(Q37-S)
- Q39 pad 1: /jk-flipflop1/NAND3_1/Out -> /jk-flipflop/NAND2_1/Out
- Q39 pad 3: /jk-flipflop1/Q -> /jk-flipflop/NAND2_3/A
- Q4 pad 1: /jk-flipflop1/J -> /jk-flipflop1/CLK
- Q4 pad 2: +3V3 -> Net-(Q4-S)
- Q4 pad 3: /jk-flipflop1/NAND3_1/Out -> /jk-flipflop1/NAND2_2/B
- Q40 pad 1: /jk-flipflop/J -> /jk-flipflop/\clk
- Q40 pad 2: Net-(Q25-D) -> +3V3
- Q40 pad 3: /jk-flipflop/NAND3_1/Out -> /jk-flipflop/NAND2_3/A
- Q41 pad 1: /jk-flipflop1/Clr -> /jk-flipflop/\clk
- Q41 pad 2: GND -> +3V3
- Q41 pad 3: Net-(Q35-S) -> /jk-flipflop/NAND2_4/B
- Q42 pad 1: /jk-flipflop/CLK -> /jk-flipflop/\clk
- Q42 pad 2: +3V3 -> Net-(Q42-S)
- Q42 pad 3: /jk-flipflop/NAND3_2/Out -> /jk-flipflop/NAND2_4/B
- Q43 pad 1: /jk-flipflop4/CLK -> /jk-flipflop/NAND2_1/B
- Q43 pad 2: +3V3 -> Net-(Q43-S)
- Q43 pad 3: /jk-flipflop4/NAND3_1/Out -> Net-(Q42-S)
- Q44 pad 1: /jk-flipflop4/Q -> /jk-flipflop/Preset
- Q44 pad 2: +3V3 -> GND
- Q44 pad 3: /jk-flipflop4/NAND3_2/Out -> Net-(Q43-S)
- Q45 pad 1: /jk-flipflop1/Q -> /jk-flipflop/NAND2_1/B
- Q45 pad 2: Net-(Q35-D) -> +3V3
- Q45 pad 3: /jk-flipflop1/\Q -> /jk-flipflop/NAND2_4/B
- Q46 pad 1: /jk-flipflop4/K -> /jk-flipflop/Preset
- Q46 pad 2: GND -> +3V3
- Q46 pad 3: Net-(Q46-D) -> /jk-flipflop/NAND2_4/B
- Q47 pad 1: /jk-flipflop4/Q -> /jk-flipflop1/\clk
- Q47 pad 2: Net-(Q46-D) -> +3V3
- Q47 pad 3: Net-(Q47-D) -> /jk-flipflop1/NAND2_4/B
- Q48 pad 1: /jk-flipflop/CLK -> /jk-flipflop1/\clk
- Q48 pad 2: Net-(Q37-D) -> Net-(Q48-S)
- Q48 pad 3: /jk-flipflop/NAND3_2/Out -> /jk-flipflop1/NAND2_4/B
- Q49 pad 1: /jk-flipflop/K -> /jk-flipflop1/NAND2_1/B
- Q49 pad 2: +3V3 -> Net-(Q49-S)
- Q49 pad 3: /jk-flipflop/NAND3_2/Out -> Net-(Q48-S)
- Q5 pad 1: /jk-flipflop1/CLK -> /jk-flipflop1/Q
- Q5 pad 2: +3V3 -> Net-(Q5-S)
- Q5 pad 3: /jk-flipflop1/NAND3_1/Out -> Net-(Q4-S)
- Q50 pad 1: /jk-flipflop/K -> /jk-flipflop1/Preset
- Q50 pad 3: Net-(Q37-S) -> Net-(Q49-S)
- Q51 pad 1: /jk-flipflop4/CLK -> /jk-flipflop1/NAND2_1/B
- Q51 pad 3: /jk-flipflop4/NAND3_2/Out -> /jk-flipflop1/NAND2_4/B
- Q52 pad 1: /jk-flipflop3/NAND3_2/Out -> /jk-flipflop1/Preset
- Q52 pad 2: Net-(Q52-S) -> +3V3
- Q52 pad 3: Net-(Q52-D) -> /jk-flipflop1/NAND2_4/B
- Q53 pad 1: /jk-flipflop1/Clr -> /jk-flipflop1/NAND2_1/Out
- Q53 pad 3: /jk-flipflop1/\Q -> /jk-flipflop1/NAND2_1/B
- Q54 pad 1: /jk-flipflop3/Clr -> /jk-flipflop1/NAND2_1/Out
- Q54 pad 2: +3V3 -> Net-(Q54-S)
- Q54 pad 3: /jk-flipflop3/\Q -> /jk-flipflop1/NAND2_1/B
- Q55 pad 1: /jk-flipflop1/Q -> /jk-flipflop1/NAND2_2/B
- Q55 pad 2: +3V3 -> GND
- Q55 pad 3: /jk-flipflop1/\Q -> Net-(Q54-S)
- Q56 pad 1: /jk-flipflop3/NAND3_2/Out -> /jk-flipflop1/NAND2_2/B
- Q56 pad 3: /jk-flipflop3/\Q -> /jk-flipflop1/NAND2_1/B
- Q57 pad 1: /jk-flipflop4/K -> /jk-flipflop4/CLK
- Q57 pad 3: /jk-flipflop4/NAND3_2/Out -> /jk-flipflop4/\clk
- Q58 pad 1: /jk-flipflop3/Q -> /jk-flipflop4/CLK
- Q58 pad 2: Net-(Q52-D) -> GND
- Q58 pad 3: /jk-flipflop3/\Q -> /jk-flipflop4/\clk
- Q59 pad 1: /jk-flipflop4/CLK -> /jk-flipflop4/Clr
- Q59 pad 2: Net-(Q47-D) -> +3V3
- Q59 pad 3: /jk-flipflop4/NAND3_2/Out -> /jk-flipflop4/NAND2_3/A
- Q6 pad 1: /jk-flipflop1/Q -> /jk-flipflop1/K
- Q6 pad 2: Net-(Q15-D) -> GND
- Q6 pad 3: Net-(Q6-D) -> Net-(Q5-S)
- Q60 pad 1: /jk-flipflop4/CLK -> /jk-flipflop4/Clr
- Q60 pad 2: GND -> Net-(Q60-S)
- Q60 pad 3: Net-(Q60-D) -> /jk-flipflop4/NAND2_3/A
- Q61 pad 1: /jk-flipflop3/Clr -> /jk-flipflop4/NAND2_1/Out
- Q61 pad 2: GND -> Net-(Q61-S)
- Q61 pad 3: Net-(Q52-S) -> Net-(Q60-S)
- Q62 pad 1: /jk-flipflop3/Q -> /jk-flipflop4/\clk
- Q62 pad 2: +3V3 -> GND
- Q62 pad 3: /jk-flipflop3/\Q -> Net-(Q61-S)
- Q63 pad 1: /jk-flipflop4/\Q -> /jk-flipflop4/NAND2_1/Out
- Q63 pad 2: Net-(Q60-D) -> +3V3
- Q63 pad 3: Net-(Q63-D) -> /jk-flipflop4/NAND2_3/A
- Q64 pad 1: /jk-flipflop4/J -> /jk-flipflop4/\clk
- Q64 pad 2: Net-(Q63-D) -> +3V3
- Q64 pad 3: /jk-flipflop4/NAND3_1/Out -> /jk-flipflop4/NAND2_3/A
- Q65 pad 1: /jk-flipflop4/J -> /jk-flipflop4/\clk
- Q65 pad 3: /jk-flipflop4/NAND3_1/Out -> /jk-flipflop4/NAND2_4/B
- Q66 pad 1: /jk-flipflop4/\Q -> /jk-flipflop4/\clk
- Q66 pad 2: +3V3 -> Net-(Q66-S)
- Q66 pad 3: /jk-flipflop4/NAND3_1/Out -> /jk-flipflop4/NAND2_4/B
- Q67 pad 1: /jk-flipflop3/\Q -> /jk-flipflop4/NAND2_1/B
- Q67 pad 2: GND -> Net-(Q67-S)
- Q67 pad 3: Net-(Q67-D) -> Net-(Q66-S)
- Q68 pad 1: /jk-flipflop3/NAND3_1/Out -> /jk-flipflop4/Preset
- Q68 pad 2: +3V3 -> GND
- Q68 pad 3: /jk-flipflop3/Q -> Net-(Q67-S)
- Q69 pad 1: /jk-flipflop3/Preset -> /jk-flipflop4/NAND2_1/B
- Q69 pad 2: Net-(Q69-S) -> +3V3
- Q69 pad 3: /jk-flipflop3/Q -> /jk-flipflop4/NAND2_4/B
- Q7 pad 1: /jk-flipflop1/J -> /jk-flipflop1/Q
- Q7 pad 2: Net-(Q2-D) -> +3V3
- Q7 pad 3: /jk-flipflop1/NAND3_1/Out -> /jk-flipflop1/NAND2_2/B
- Q70 pad 1: /jk-flipflop3/\Q -> /jk-flipflop4/Preset
- Q70 pad 3: /jk-flipflop3/Q -> /jk-flipflop4/NAND2_4/B
- Q71 pad 1: /jk-flipflop3/Preset -> /jk-flipflop4/J
- Q71 pad 3: /jk-flipflop3/Q -> /jk-flipflop4/NAND2_1/A
- Q72 pad 1: /jk-flipflop3/NAND3_1/Out -> /jk-flipflop4/J
- Q72 pad 2: Net-(Q67-D) -> Net-(Q72-S)
- Q72 pad 3: Net-(Q69-S) -> /jk-flipflop4/NAND2_1/A
- Q73 pad 1: /jk-flipflop/\Q -> /jk-flipflop4/\Q
- Q73 pad 2: +3V3 -> Net-(Q73-S)
- Q73 pad 3: /jk-flipflop/Q -> Net-(Q72-S)
- Q74 pad 1: /jk-flipflop/NAND3_1/Out -> /jk-flipflop4/CLK
- Q74 pad 2: +3V3 -> GND
- Q74 pad 3: /jk-flipflop/Q -> Net-(Q73-S)
- Q75 pad 1: /jk-flipflop/Preset -> /jk-flipflop4/\Q
- Q75 pad 3: /jk-flipflop/Q -> /jk-flipflop4/NAND2_1/A
- Q76 pad 1: /jk-flipflop/NAND3_1/Out -> /jk-flipflop4/CLK
- Q76 pad 2: Net-(Q76-S) -> +3V3
- Q76 pad 3: Net-(Q76-D) -> /jk-flipflop4/NAND2_1/A
- Q77 pad 1: /jk-flipflop/NAND3_2/Out -> /jk-flipflop3/CLK
- Q77 pad 2: Net-(Q77-S) -> +3V3
- Q77 pad 3: Net-(Q77-D) -> /jk-flipflop3/\clk
- Q78 pad 1: /jk-flipflop/\Q -> /jk-flipflop3/CLK
- Q78 pad 3: Net-(Q76-S) -> /jk-flipflop3/\clk
- Q79 pad 1: /jk-flipflop/NAND3_2/Out -> /jk-flipflop3/CLK
- Q79 pad 3: /jk-flipflop/\Q -> /jk-flipflop3/NAND2_2/B
- Q8 pad 1: /jk-flipflop1/\Q -> /jk-flipflop1/K
- Q8 pad 3: /jk-flipflop1/NAND3_1/Out -> /jk-flipflop1/NAND2_2/B
- Q80 pad 1: /jk-flipflop/Preset -> /jk-flipflop3/CLK
- Q80 pad 2: Net-(Q76-D) -> Net-(Q80-S)
- Q80 pad 3: /jk-flipflop/Q -> /jk-flipflop3/NAND2_2/B
- Q81 pad 1: /jk-flipflop3/CLK -> /jk-flipflop3/Q
- Q81 pad 3: /jk-flipflop3/NAND3_2/Out -> Net-(Q80-S)
- Q82 pad 1: /jk-flipflop/Clr -> /jk-flipflop3/K
- Q82 pad 2: +3V3 -> GND
- Q82 pad 3: /jk-flipflop/\Q -> Net-(Q81-S)
- Q83 pad 2: Net-(Q83-S) -> +3V3
- Q83 pad 3: Net-(Q81-S) -> /jk-flipflop3/NAND2_2/B
- Q84 pad 1: /jk-flipflop3/CLK -> /jk-flipflop3/K
- Q84 pad 3: /jk-flipflop3/NAND3_2/Out -> /jk-flipflop3/NAND2_2/B
- Q85 pad 1: /jk-flipflop3/Q -> /jk-flipflop3/J
- Q85 pad 3: /jk-flipflop3/NAND3_2/Out -> /jk-flipflop3/NAND2_1/A
- Q86 pad 1: /jk-flipflop3/K -> /jk-flipflop3/J
- Q86 pad 2: GND -> Net-(Q86-S)
- Q86 pad 3: Net-(Q83-S) -> /jk-flipflop3/NAND2_1/A
- Q87 pad 1: /jk-flipflop3/K -> /jk-flipflop3/\Q
- Q87 pad 2: +3V3 -> Net-(Q87-S)
- Q87 pad 3: /jk-flipflop3/NAND3_2/Out -> Net-(Q86-S)
- Q88 pad 1: /jk-flipflop/Clr -> /jk-flipflop3/CLK
- Q88 pad 3: Net-(Q77-S) -> Net-(Q87-S)
- Q89 pad 1: /jk-flipflop/Q -> /jk-flipflop3/\Q
- Q89 pad 3: /jk-flipflop/\Q -> /jk-flipflop3/NAND2_1/A
- Q9 pad 1: /jk-flipflop1/CLK -> /jk-flipflop1/J
- Q9 pad 2: Net-(Q6-D) -> +3V3
- Q9 pad 3: /jk-flipflop1/NAND3_2/Out -> /jk-flipflop1/NAND2_1/A
- Q90 pad 1: /jk-flipflop/Q -> /jk-flipflop3/CLK
- Q90 pad 2: Net-(Q77-D) -> +3V3
- Q90 pad 3: /jk-flipflop/\Q -> /jk-flipflop3/NAND2_1/A
- Q91 pad 1: /jk-flipflop3/\Q -> /jk-flipflop3/Clr
- Q91 pad 2: Net-(Q91-S) -> +3V3
- Q91 pad 3: Net-(Q91-D) -> /jk-flipflop3/NAND2_3/A
- Q92 pad 1: /jk-flipflop3/J -> /jk-flipflop3/Clr
- Q92 pad 2: Net-(Q91-D) -> Net-(Q92-S)
- Q92 pad 3: /jk-flipflop3/NAND3_1/Out -> /jk-flipflop3/NAND2_3/A
- Q93 pad 1: /jk-flipflop3/J -> /jk-flipflop3/NAND2_1/Out
- Q93 pad 2: +3V3 -> Net-(Q93-S)
- Q93 pad 3: /jk-flipflop3/NAND3_1/Out -> Net-(Q92-S)
- Q94 pad 1: /jk-flipflop3/CLK -> /jk-flipflop3/\clk
- Q94 pad 2: +3V3 -> GND
- Q94 pad 3: /jk-flipflop3/NAND3_1/Out -> Net-(Q93-S)
- Q95 pad 1: /jk-flipflop3/CLK -> /jk-flipflop3/NAND2_1/Out
- Q95 pad 2: GND -> +3V3
- Q95 pad 3: Net-(Q91-S) -> /jk-flipflop3/NAND2_3/A
- Q96 pad 1: /jk-flipflop3/\Q -> /jk-flipflop3/\clk
- Q96 pad 3: /jk-flipflop3/NAND3_1/Out -> /jk-flipflop3/NAND2_3/A
Routing:
- net /jk-flipflop4/Q: track 104.3 -> 16.3 mm, vias 3 -> 0
- net /jk-flipflop3/Q: track 87.4 -> 16.3 mm, vias 3 -> 0
- net /jk-flipflop4/Preset: track 74.8 -> 4.36 mm, vias 2 -> 0
- net /jk-flipflop4/\Q: track 90.8 -> 24.1 mm, vias 3 -> 0
- net GND: track 83.6 -> 17.3 mm, vias 4 -> 16
- net /jk-flipflop3/J: track 71.6 -> 8.50 mm, vias 2 -> 0
- net /jk-flipflop3/Preset: track 67.2 -> 4.36 mm, vias 2 -> 0
- net /jk-flipflop3/CLK: track 72.8 -> 12.9 mm, vias 3 -> 0
- net /jk-flipflop4/J: track 64.4 -> 8.50 mm, vias 2 -> 0
- net /jk-flipflop3/\Q: track 78.9 -> 24.1 mm, vias 2 -> 0
- net /jk-flipflop4/CLK: track 65.3 -> 12.9 mm, vias 3 -> 0
- net /jk-flipflop3/K: track 56.2 -> 4.36 mm, vias 2 -> 0
- net /jk-flipflop4/Clr: track 57.0 -> 8.50 mm
- net /jk-flipflop1/K: track 50.1 -> 4.36 mm, vias 1 -> 0
- net /jk-flipflop/Q: track 61.2 -> 16.3 mm, vias 4 -> 0
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
Commit message: flipflop routing wip
Parts:
- added C5: 100n, Capacitor_SMD:C_0603_1608Metric, F.Cu at (116.5, 54.8)
- added C6: 100n, Capacitor_SMD:C_0603_1608Metric, F.Cu at (90.5, 54.8)
- added C7: 100n, Capacitor_SMD:C_0603_1608Metric, F.Cu at (64.1, 77.2)
- added C8: 100n, Capacitor_SMD:C_0603_1608Metric, F.Cu at (167.0, 116.8)
- moved Q47 355.0 mm to (106.6, 56.7), turned to 90 degrees
- moved Q48 353.3 mm to (110.1, 56.6), turned to 90 degrees
- moved Q51 351.5 mm to (113.6, 56.7), turned to 90 degrees
- moved Q52 349.6 mm to (106.6, 60.8), turned to 90 degrees
- moved Q50 347.8 mm to (110.1, 60.8), turned to 90 degrees
- moved Q49 346.1 mm to (113.6, 60.8), turned to 90 degrees
- moved Q125 332.7 mm to (120.5, 47.1)
- moved Q126 332.7 mm to (120.5, 50.6)
- moved Q127 332.7 mm to (124.6, 50.6)
- moved Q128 332.7 mm to (124.6, 47.1)
- moved Q162 326.9 mm to (79.3, 90.0)
- moved Q161 326.9 mm to (79.2, 86.5)
- moved Q163 326.9 mm to (83.4, 90.0)
- moved Q164 326.9 mm to (83.4, 86.5)
- moved Q79 322.8 mm to (66.7, 85.8), turned to 90 degrees
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Connections:
- Q100 pad 1: /jk-flipflop3/Preset -> /jk-flipflop3/\clk
- Q102 pad 1: /jk-flipflop3/Preset -> /jk-flipflop3/\clk
- Q103 pad 1: /jk-flipflop4/CLK -> /jk-flipflop4/K
- Q105 pad 1: /jk-flipflop4/CLK -> /jk-flipflop4/K
- Q107 pad 1: /jk-flipflop4/K -> /jk-flipflop4/CLK
- Q112 pad 1: /jk-flipflop4/K -> /jk-flipflop4/CLK
- Q29 pad 1: /jk-flipflop/CLK -> /jk-flipflop/K
- Q3 pad 1: /jk-flipflop1/CLK -> /jk-flipflop1/K
- Q30 pad 1: /jk-flipflop/CLK -> /jk-flipflop/K
- Q32 pad 1: /jk-flipflop/K -> /jk-flipflop/CLK
- Q34 pad 1: /jk-flipflop/K -> /jk-flipflop/CLK
- Q4 pad 1: /jk-flipflop1/CLK -> /jk-flipflop1/K
- Q41 pad 1: /jk-flipflop/\clk -> /jk-flipflop/Preset
- Q42 pad 1: /jk-flipflop/\clk -> /jk-flipflop/Preset
- Q44 pad 1: /jk-flipflop/Preset -> /jk-flipflop/\clk
- Q46 pad 1: /jk-flipflop/Preset -> /jk-flipflop/\clk
- Q47 pad 1: /jk-flipflop1/\clk -> /jk-flipflop1/Preset
- Q48 pad 1: /jk-flipflop1/\clk -> /jk-flipflop1/Preset
- Q50 pad 1: /jk-flipflop1/Preset -> /jk-flipflop1/\clk
- Q52 pad 1: /jk-flipflop1/Preset -> /jk-flipflop1/\clk
- Q6 pad 1: /jk-flipflop1/K -> /jk-flipflop1/CLK
- Q65 pad 1: /jk-flipflop4/\clk -> /jk-flipflop4/Preset
- Q66 pad 1: /jk-flipflop4/\clk -> /jk-flipflop4/Preset
- Q68 pad 1: /jk-flipflop4/Preset -> /jk-flipflop4/\clk
- Q70 pad 1: /jk-flipflop4/Preset -> /jk-flipflop4/\clk
- Q79 pad 1: /jk-flipflop3/CLK -> /jk-flipflop3/K
- Q8 pad 1: /jk-flipflop1/K -> /jk-flipflop1/CLK
- Q80 pad 1: /jk-flipflop3/CLK -> /jk-flipflop3/K
- Q82 pad 1: /jk-flipflop3/K -> /jk-flipflop3/CLK
- Q84 pad 1: /jk-flipflop3/K -> /jk-flipflop3/CLK
- Q97 pad 1: /jk-flipflop3/\clk -> /jk-flipflop3/Preset
- Q98 pad 1: /jk-flipflop3/\clk -> /jk-flipflop3/Preset
Routing:
- net /jk-flipflop4/\Q: track 24.1 -> 87.0 mm, vias 0 -> 3
- net /jk-flipflop1/\Q: track 24.1 -> 87.0 mm, vias 0 -> 3
- net /jk-flipflop/\Q: track 24.1 -> 87.0 mm, vias 0 -> 3
- net /jk-flipflop/Q: track 16.3 -> 70.8 mm, vias 0 -> 2
- net /jk-flipflop1/Q: track 16.3 -> 70.8 mm, vias 0 -> 2
- net /jk-flipflop4/Q: track 16.3 -> 70.8 mm, vias 0 -> 2
- net /jk-flipflop3/NAND2_1/Out: track 16.3 -> 62.7 mm, vias 0 -> 4
- net /jk-flipflop3/\Q: track 24.1 -> 66.2 mm, vias 0 -> 3
- net /jk-flipflop3/\clk: track 12.9 -> 44.4 mm, vias 0 -> 2
- net /jk-flipflop3/NAND2_1/B: track 24.1 -> 55.5 mm, vias 0 -> 3
- net /jk-flipflop3/CLK: track 12.9 -> 44.1 mm
- net /jk-flipflop3/Q: track 16.3 -> 46.0 mm, vias 0 -> 3
- net /jk-flipflop3/NAND2_3/A: track 15.7 -> 42.5 mm, vias 0 -> 2
- net /jk-flipflop3/NAND2_2/B: track 23.5 -> 47.5 mm, vias 0 -> 4
- net /jk-flipflop/CLK: track 12.9 -> 33.9 mm
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- added copper zone on In1.Cu, net +3V3
- added copper zone on In2.Cu, net GND
- removed copper zone on B.Cu, net +3V3
- removed copper zone on F.Cu, net GND
Other:
- board size 57.2 x 61.2 mm -> 80 x 61.2 mm
- copper layers 2 -> 4

Commit message: routed flipflops
Connections:
- J1 pad 12: /jk-flipflop/J -> /jk-flipflop1/J
- J1 pad 14: /jk-flipflop/CLK -> /jk-flipflop1/CLK
- J1 pad 16: /jk-flipflop/K -> /jk-flipflop1/K
- J1 pad 2: /jk-flipflop/Clr -> /jk-flipflop1/Clr
- J1 pad 20: /jk-flipflop1/Clr -> /jk-flipflop3/Clr
- J1 pad 21: /jk-flipflop3/J -> /jk-flipflop/J
- J1 pad 22: /jk-flipflop1/Q -> /jk-flipflop3/\Q
- J1 pad 23: /jk-flipflop3/CLK -> /jk-flipflop/CLK
- J1 pad 24: /jk-flipflop1/\Q -> /jk-flipflop3/Q
- J1 pad 25: /jk-flipflop3/K -> /jk-flipflop/K
- J1 pad 26: /jk-flipflop1/Preset -> /jk-flipflop3/Preset
- J1 pad 29: /jk-flipflop3/Clr -> /jk-flipflop/Clr
- J1 pad 30: /jk-flipflop1/J -> /jk-flipflop3/J
- J1 pad 31: /jk-flipflop3/\Q -> /jk-flipflop/Q
- J1 pad 32: /jk-flipflop1/CLK -> /jk-flipflop3/CLK
- J1 pad 33: /jk-flipflop3/Q -> /jk-flipflop/\Q
- J1 pad 34: /jk-flipflop1/K -> /jk-flipflop3/K
- J1 pad 35: /jk-flipflop3/Preset -> /jk-flipflop/Preset
- J1 pad 4: /jk-flipflop/Q -> /jk-flipflop1/Q
- J1 pad 6: /jk-flipflop/\Q -> /jk-flipflop1/\Q
- J1 pad 8: /jk-flipflop/Preset -> /jk-flipflop1/Preset
Routing:
- net /jk-flipflop3/J: track 8.50 -> 107.9 mm, vias 0 -> 1
- net /jk-flipflop3/K: track 10.00 -> 95.9 mm
- net /jk-flipflop4/J: track 8.50 -> 84.2 mm, vias 0 -> 2
- net /jk-flipflop3/CLK: track 44.1 -> 108.7 mm, vias 0 -> 1
- net /jk-flipflop3/Clr: track 8.50 -> 68.8 mm
- net /jk-flipflop4/CLK: track 33.9 -> 94.0 mm, vias 0 -> 2
- net /jk-flipflop/J: track 8.50 -> 68.1 mm, vias 0 -> 2
- net /jk-flipflop3/Q: track 46.0 -> 103.1 mm, vias 3 -> 4
- net /jk-flipflop3/\Q: track 66.2 -> 123.2 mm, vias 3 -> 4
- net /jk-flipflop3/Preset: track 8.50 -> 62.5 mm, vias 0 -> 1
- net /jk-flipflop4/Preset: track 8.50 -> 58.6 mm
- net /jk-flipflop/CLK: track 33.9 -> 77.6 mm, vias 0 -> 2
- net /jk-flipflop1/CLK: track 33.9 -> 76.0 mm, vias 0 -> 1
- net /jk-flipflop4/K: track 22.7 -> 64.5 mm, vias 1 -> 2
- net /jk-flipflop1/K: track 22.7 -> 64.3 mm
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
Commit message: updated production files
Routing:
- net +3V3: track 75.1 -> 89.8 mm, vias 80 -> 85
- net GND: track 35.8 -> 48.5 mm, vias 38 -> 43

Commit message: forgot to caps on flipflop module
Parts:
- moved C8 59.9 mm to (110.3, 97.4)
- moved C4 55.5 mm to (110.3, 95.7)
Routing:
- net +3V3: track 89.8 -> 91.8 mm, vias 85 -> 87
- net GND: track 48.5 -> 50.4 mm, vias 43 -> 45
Changed lines of the file:
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@@
 	(footprint "Capacitor_SMD:C_0603_1608Metric"
 		(layer "F.Cu")
-		(at 161.825 116.2 180)
+		(at 110.3 95.65 180)
 		(descr "Capacitor SMD 0603 (1608 Metric), square (rectangular) end terminal, IPC-7351 nominal, (Body size source: IPC-SM-782 page 76, https://www.pcb-3d.com/wordpress/wp-content/uploads/ipc-sm-782a_amendment_1_and_2.pdf), generated with kicad-footprint-generator")
 		(tags "capacitor")
@@
 	(footprint "Capacitor_SMD:C_0603_1608Metric"
 		(layer "F.Cu")
-		(at 167 116.85)
+		(at 110.3 97.4)
 		(descr "Capacitor SMD 0603 (1608 Metric), square (rectangular) end terminal, IPC-7351 nominal, (Body size source: IPC-SM-782 page 76, https://www.pcb-3d.com/wordpress/wp-content/uploads/ipc-sm-782a_amendment_1_and_2.pdf), generated with kicad-footprint-generator")
 		(tags "capacitor")
 		(property "Reference" "C8"
-			(at -2.0825 0 0)
+			(at -2.675 0 0)
 			(layer "F.SilkS")
 			(effects
@@
 	)
 	(segment
+		(start 112.1 95.65)
+		(end 112.125 95.675)
+		(width 0.2)
+		(layer "F.Cu")
+		(net 1)
+	)
+	(segment
 		(start 85.225 48.6525)
 		(end 85.86 49.2875)
@@
 	)
 	(segment
+		(start 109.525 97.4)
+		(end 109.525 98.325)
+		(width 0.2)
+		(layer "F.Cu")
+		(net 1)
+	)
+	(segment
 		(start 91.6 95.7)
 		(end 91.6 95.695)
@@
 	)
 	(segment
+		(start 111.075 95.65)
+		(end 112.1 95.65)
+		(width 0.2)
+		(layer "F.Cu")
+		(net 1)
+	)
+	(segment
 		(start 59.16 48.565)
 		(end 59.795 49.2)
@@
 	)
 	(via
+		(at 112.125 95.675)
+		(size 0.4)
+		(drill 0.3)
+		(layers "F.Cu" "B.Cu")
+		(net 1)
+	)
+	(via
 		(at 124.2775 48.6525)
 		(size 0.4)
@@
 	)
 	(via
+		(at 109.525 98.325)
+		(size 0.4)
+		(drill 0.3)
+		(layers "F.Cu" "B.Cu")
+		(net 1)
+	)
+	(via
 		(at 102.675 41.625)
 		(size 0.4)
@@
 	)
 	(segment
+		(start 111.075 98.3)
+		(end 111.025 98.35)
+		(width 0.2)
+		(layer "F.Cu")
+		(net 2)
+	)
+	(segment
 		(start 123.96 51.1925)
 		(end 123.96 50.5625)
@@
 	)
 	(segment
+		(start 109.525 95.65)
+		(end 108.55 95.65)
+		(width 0.2)
+		(layer "F.Cu")
+		(net 2)
+	)
+	(segment
 		(start 92.35 40.005)
 		(end 92.35 41.075)
@@
 	)
 	(segment
+		(start 111.075 97.4)
+		(end 111.075 98.3)
+		(width 0.2)
+		(layer "F.Cu")
+		(net 2)
+	)
+	(segment
 		(start 84.5525 61.2775)
 		(end 84.455 61.2775)
@@
 	)
 	(via
+		(at 111.025 98.35)
+		(size 0.4)
+		(drill 0.3)
+		(layers "F.Cu" "B.Cu")
+		(net 2)
+	)
+	(via
 		(at 71.86 50.475)
 		(size 0.4)
 		(drill 0.3)
+		(layers "F.Cu" "B.Cu")
+		(net 2)
+	)
+	(via
+		(at 108.55 95.65)
+		(size 0.4)
+		(drill 0.3)
